File: estabilizador.sch (KiCad schematic (older format))
At the start: 91 parts, among them J1 Tensão de Entrada, J10 Driver, J11 Tensão do Estágio de Reles, J12 Tensão do Estágio do Inversor, J13 Tensão de Saída Total, J14 Tensão de Medição, J15 Tap AUX2, J2 Autotransformador, J3 Comandos Reles, J4 Tap AUX1, J5 Comandos PWMs, J6 Fonte Aux, J7 Driver, J8 Driver, J9 Driver, K1 RT42xxxx, K2 RT42xxxx, K3 RT42xxxx, Q1 BC517, Q2 BC517, Q3 IRF840N, Q4 IRF840N, Q5 BC517, Q6 IRF840N, Q7 IRF840N, U1 LV20-P, U2 LV25-P

Commit message: Modificação do esquemático
Parts:
- removed C1, C2: 1000uF, Capacitor_THT:CP_Radial_D18.0mm_P7.50mm, symbol Device:CP1_Small
- removed C12, C13: 2uF, Capacitor_THT:C_Rect_L29.0mm_W7.6mm_P27.50mm_MKT, symbol Device:C_Small
- removed C14, C15: 1uF, Capacitor_THT:C_Rect_L29.0mm_W7.6mm_P27.50mm_MKT, symbol Device:C_Small
- removed D1: GBU8J, Diode_THT:Diode_Bridge_Vishay_KBU, symbol Diode_Bridge:GBU8J
- removed D2, D3, D4: 1N4148, Diode_THT:D_DO-35_SOD27_P7.62mm_Horizontal, symbol Diode:1N4148
- removed J15: Tap AUX2, Connector_Phoenix_MSTB:PhoenixContact_MSTBVA_2,5_4-G-5,08_1x04_P5.08mm_Vertical, symbol Connector:Screw_Terminal_01x04
- removed J2: Autotransformador, Connector_Phoenix_MSTB:PhoenixContact_MSTBVA_2,5_5-G-5,08_1x05_P5.08mm_Vertical, symbol Connector:Screw_Terminal_01x05
- removed J3: Comandos Reles, Connector_PinHeader_2.54mm:PinHeader_1x06_P2.54mm_Vertical, symbol Connector_Generic:Conn_01x06
- removed JP8, JP9: Jumper_NO_Small, Connector_PinHeader_2.54mm:PinHeader_1x02_P2.54mm_Vertical, symbol Device:Jumper_NO_Small
- removed K1: RT42xxxx, Relay:Relay_DPDT_model_A, symbol Relay:RT42xxxx
- removed K2, K3: RT42xxxx, Relay:Relay_DPDT_model_B, symbol Relay:RT42xxxx
- removed Q1, Q2, Q5: BC517, Package_TO_SOT_THT:TO-92_Inline_Wide, symbol Transistor_BJT:BC517
- removed R14, R16: 10k, Resistor_THT:R_Axial_DIN0414_L11.9mm_D4.5mm_P15.24mm_Horizontal, symbol Device:R_US
- removed R21, R22, R23: 10K, Resistor_SMD:R_0805_2012Metric_Pad1.15x1.40mm_HandSolder, symbol Device:R_US
- added D1: 3,3 V, Diode_SMD:D_SOT-23_ANK, symbol Device:D_Zener
- added J15: Comandos PWMs, Connector_PinHeader_2.54mm:PinHeader_1x08_P2.54mm_Vertical, symbol Connector_Generic:Conn_01x08
- added J16, J17, J18, J19: Driver, Connector_PinHeader_2.54mm:PinHeader_1x07_P2.54mm_Vertical, symbol Connector:Conn_01x07_Female
- added J2: Alimentação ACS712, Connector_PinHeader_2.54mm:PinHeader_1x02_P2.54mm_Vertical, symbol Connector_Generic:Conn_01x02
- added J21: Conn_01x03_Female, Connector_PinHeader_2.54mm:PinHeader_1x03_P2.54mm_Vertical, symbol Connector:Conn_01x03_Female
- added J23: Medição da Corrente, Connector_PinHeader_2.54mm:PinHeader_1x02_P2.54mm_Vertical, symbol Connector_Generic:Conn_01x02
- added J4: Screw_Terminal_01x02, Connector_Phoenix_MSTB:PhoenixContact_MSTBVA_2,5_2-G-5,08_1x02_P5.08mm_Vertical, symbol Connector:Screw_Terminal_01x02
- added J5: Sensor de Corrente, Connector_Phoenix_MSTB:PhoenixContact_MSTBVA_2,5_2-G-5,08_1x02_P5.08mm_Vertical, symbol Connector:Screw_Terminal_01x02
- added J9: Tensão de Saída do Boost, Connector_Phoenix_MSTB:PhoenixContact_MSTBVA_2,5_2-G-5,08_1x02_P5.08mm_Vertical, symbol Connector:Screw_Terminal_01x02
- added L1: L_Core_Ferrite, boost_pfc:NEE_30-14, symbol Device:L_Core_Ferrite
- added Q1, Q2, Q3, Q4: IRG4PF50W, Package_TO_SOT_THT:TO-247-3_Vertical, symbol Transistor_IGBT:IRG4PF50W
- added R17: 567, Resistor_SMD:R_0805_2012Metric_Pad1.15x1.40mm_HandSolder, symbol Device:R_US
- added R2: 10k, Resistor_SMD:R_0805_2012Metric_Pad1.15x1.40mm_HandSolder, symbol Device:R_US
- added R27, R28, R29, R30, R31, R32, R33, R34: 340R, Resistor_SMD:R_1206_3216Metric_Pad1.42x1.75mm_HandSolder, symbol Device:R_US
- added TP10, TP11, TP12, TP13, TP14, TP15, TP16, TP9: TestPoint, Connector_PinHeader_2.54mm:PinHeader_1x01_P2.54mm_Vertical, symbol estabilizador-rescue:TestPoint-Connector
- C1: renamed from C3; value 1000uF -> 2700uF
- J6: renamed from J11; value Tensão do Estágio de Reles -> Tensão do Estabilizador
- L2: renamed from L1; footprint Inductors:Inductor_EE4220 -> boost_pfc:NEE_45-45
- Q5: renamed from Q3; footprint transistors:TO-220-3 Heatsink -> boost_pfc:TO-220-3 Heatsink
- Q6: footprint transistors:TO-220-3 Heatsink -> boost_pfc:TO-220-3 Heatsink
- Q7: renamed from Q4; footprint transistors:TO-220-3 Heatsink -> boost_pfc:TO-220-3 Heatsink
- Q8: renamed from Q7; footprint transistors:TO-220-3 Heatsink -> boost_pfc:TO-220-3 Heatsink
- R1, R3, R5: value 100K -> 10k
- R15: renamed from R9; footprint Resistor_THT:R_Axial_DIN0414_L11.9mm_D4.5mm_P15.24mm_Horizontal -> Resistor_THT:R_Axial_DIN0207_L6.3mm_D2.5mm_P10.16mm_Horizontal
- R16: renamed from R12; footprint Resistor_THT:R_Axial_DIN0414_L11.9mm_D4.5mm_P15.24mm_Horizontal -> Resistor_THT:R_Axial_DIN0207_L6.3mm_D2.5mm_P10.16mm_Horizontal
- renumbered C8 to C10, C9 to C11, C10 to C12, C11 to C13, C4 to C6, C6 to C8, C5 to C9, J5 to J10, J7 to J11, J8 to J12, J9 to J13, J10 to J14, J6 to J20, J14 to J22, J4 to J3, J12 to J7, J13 to J8, JP4 to JP3, JP3 to JP4, R11 to R10, R8 to R11, R10 to R12, R15 to R14, R17 to R19, R2 to R20, R18 to R21, R4 to R22, R19 to R23, R6 to R24, R20 to R25, R7 to R26, R24 to R6, R25 to R7, R26 to R8, R27 to R9, TP7 to TP1, TP8 to TP2, TP5 to TP3, TP6 to TP4, TP3 to TP5, TP4 to TP6, TP1 to TP7, TP2 to TP8
Connections:
- net LO_in_inv is gone; now on net Source3: C1.2, JP2.2
- net RL1 is gone; now on net Source1: R1.2
- net RL2 is gone; now on net Source3: R3.2
- net RL3 is gone; now on net Source3: R5.2
- net VauxB is gone; now on net Source2: J3.2 (Pin_2)
- net +12V: now also J16.5 (Pin_5), J17.5 (Pin_5), J18.5 (Pin_5), J19.5 (Pin_5), R27.1, R28.1, R29.1, R30.1, R31.1, R32.1, R33.1, R34.1
- net GNDREF: now also D1.2 (A), J15.2 (Pin_2), J15.4 (Pin_4), J15.6 (Pin_6), J15.8 (Pin_8), J16.4 (Pin_4), J16.7 (Pin_7), J17.4 (Pin_4), J17.7 (Pin_7), J18.4 (Pin_4), J18.7 (Pin_7), J19.4 (Pin_4), J19.7 (Pin_7), J2.2 (Pin_2), J21.3 (Pin_3), J23.2 (Pin_2)
- net Gate1: now also R1.1, Q1.1 (G); no longer Q5.1 (G), R6.1
- net Gate2: now also Q2.1 (G), R2.1; no longer Q6.1 (G), R8.1
- net Gate3: now also R3.1, Q3.1 (G); no longer Q7.1 (G), R7.1
- net Gate4: now also R5.1, Q4.1 (G); no longer Q8.1 (G), R9.1
- net NEUT: no longer U2.3 (HV-)
- net Source1: now also J5.2 (Pin_2), Q1.3 (E), Q3.2 (C); no longer L2.1, Q5.3 (S), Q7.2 (D), R6.2
- net Source2: now also Q2.3 (E), Q4.2 (C), R2.2; no longer C7.2, C8.2, C9.2, J7.2 (Pin_2), J8.1 (Pin_1), JP6.3 (B), Q6.3 (S), Q8.2 (D), R11.2, R8.2
- net Source3: now also J11.2 (Pin_2), TP7.1, U2.3 (HV-), J9.2 (Pin_2), Q3.3 (E), Q4.3 (E); no longer JP2.1, Q7.3 (S), R7.2
- net VauxA: now also L1.2
- net VtapOut: now also J1.2 (Pin_2)
- net at Q6.2 (D): now also JP1.1, Q5.2 (D), J4.1 (Pin_1)
- net at U2.1 (HV+): now also R16.1
- net HI_in_inv renamed Vboost+
- net Vboost+: now also R15.2, J9.1 (Pin_1), Q1.2 (C), Q2.2 (C)
- removed net LINE: J1.2 (Pin_2), R15.2
- net Source4 renamed Source7
- net Source7: now also JP2.1, Q7.3 (S), R7.2, J16.2 (Pin_2), J17.2 (Pin_2), J4.2 (Pin_2), TP13.1, TP15.1; no longer J11.2 (Pin_2), TP7.1
- net Vm_in renamed Vm_boost
- new net: J5.1 (Pin_1), L1.1
- new net: J21.2 (Pin_2), R17.2
- new net +5V: J2.1 (Pin_1), J21.1 (Pin_1)
- new net Gate5: J19.1 (Pin_1), Q5.1 (G), R6.1, TP10.1
- new net Gate6: J18.1 (Pin_1), Q6.1 (G), R8.1, TP12.1
- new net Gate7: J17.1 (Pin_1), Q7.1 (G), R7.1, TP14.1
- new net Gate8: J16.1 (Pin_1), Q8.1 (G), R9.1, TP16.1
- new net PWM5: J15.1 (Pin_1), J19.6 (Pin_6), R33.2, R34.2
- new net PWM6: J15.3 (Pin_3), J18.6 (Pin_6), R31.2, R32.2
- new net PWM7: J15.5 (Pin_5), J17.6 (Pin_6), R29.2, R30.2
- new net PWM8: J15.7 (Pin_7), J16.6 (Pin_6), R27.2, R28.2
- new net Source5: J19.2 (Pin_2), L2.1, Q5.3 (S), Q7.2 (D), R6.2, TP9.1
- new net Source6: C7.2, C8.2, C9.2, J18.2 (Pin_2), J7.2 (Pin_2), J8.1 (Pin_1), JP6.3 (B), Q6.3 (S), Q8.2 (D), R11.2, R8.2, TP11.1
- new net Vm_acs712: D1.1 (K), J23.1 (Pin_1), R17.1
Other:
- note removed: "180V"
- note removed: "206V"
- note removed: "220V"
- note removed: "235V"
- note removed: "41V"
- note removed: "GND"
- moved on the sheet: C1, C10, C11, C12, C13, C6, C7, C8, C9, J1, J10, J11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
