File: estabilizador.sch (KiCad schematic (older format))
At the start: 100 parts, among them J1 Tensão de Entrada, J10 Comandos PWMs, J11 Driver, J12 Driver, J13 Driver, J14 Driver, J15 Comandos PWMs, J16 Driver, J17 Driver, J18 Driver, J19 Driver, J20 Fonte Aux, J21 Alimentação LTSP 25-NP, J22 Tensão de Medição, J23 Medição da Corrente, J3 Tap AUX1, J4 Screw_Terminal_01x02, J6 Tensão do Estabilizador, J7 Tensão do Estágio do Inversor, J8 Tensão de Saída Total, J9 Tensão de Saída do Boost, Q1 IRG4PF50W, Q2 IRG4PF50W, Q3 IRG4PF50W, Q4 IRG4PF50W, Q5 IRF840N, Q6 IRF840N, Q7 IRF840N, Q8 IRF840N, U1 LV20-P, U2 LV25-P

Commit message: Modificação do esquemático
Parts:
- removed J22: Tensão de Medição, Connector_PinHeader_2.54mm:PinHeader_1x04_P2.54mm_Vertical, symbol Connector_Generic:Conn_01x04
- removed J23: Medição da Corrente, Connector_PinHeader_2.54mm:PinHeader_1x02_P2.54mm_Vertical, symbol Connector_Generic:Conn_01x02
- added C14: 100nF, Capacitor_SMD:C_0805_2012Metric_Pad1.15x1.40mm_HandSolder, symbol Device:C_Small
- added C15: 100uF, Capacitor_SMD:CP_Elec_8x10, symbol Device:CP1_Small
- added J20: Tensão de Medição, symbol Connector_Generic:Conn_01x08
- added R15, R16: 10K, Resistor_THT:R_Axial_DIN0414_L11.9mm_D4.5mm_P15.24mm_Horizontal, symbol Device:R_US
- added R19, R20: 10K, Resistor_THT:R_Axial_DIN0207_L6.3mm_D2.5mm_P10.16mm_Horizontal, symbol Device:R_US
- added U4: LV25-P, Sensor_Voltage:LEM_LV25-P, symbol Sensor_Voltage:LV25-P
- R17: renamed from R15; footprint Resistor_THT:R_Axial_DIN0207_L6.3mm_D2.5mm_P10.16mm_Horizontal -> Resistor_THT:R_Axial_DIN0414_L11.9mm_D4.5mm_P15.24mm_Horizontal
- R18: renamed from R16; footprint Resistor_THT:R_Axial_DIN0207_L6.3mm_D2.5mm_P10.16mm_Horizontal -> Resistor_THT:R_Axial_DIN0414_L11.9mm_D4.5mm_P15.24mm_Horizontal
- gave numbers to parts that had none: 1
- renumbered J15 to J10, J16 to J15, J17 to J16, J18 to J17, J19 to J18, J20 to J19, J21 to J2, J6 to J5, J7 to J6, J8 to J7, J9 to J8, J10 to J9, R19 to R21, R20 to R22, R21 to R23, R22 to R24, R23 to R25, R24 to R26, R25 to R27, R26 to R28, R27 to R29, R28 to R30, R29 to R31, R30 to R32, R31 to R33, R32 to R34, R33 to R35, R34 to R36, R34 to R37, R35 to R38
Connections:
- net labels added: Vm_tapOut
- wire segments 360 -> 380
Other:
- moved on the sheet: J10, J11, J12, J13, J14, J15, J16, J17, J18, J19, J9, JP7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

Commit message: Modificação da PCB
Parts:
- J20: footprint (none) -> Connector_PinHeader_2.54mm:PinHeader_1x08_P2.54mm_Vertical
- R38: footprint Resistor_SMD:R_0805_2012Metric_Pad1.15x1.40mm_HandSolder -> Resistor_THT:R_Axial_DIN0207_L6.3mm_D2.5mm_P10.16mm_Horizontal
Changed lines of the file:
@@
 Wire Wire Line
 	3800 2350 3800 2450
-$Comp
-L Device:R_US R37
-U 1 1 5E82D06B
-P 4350 1200
-F 0 "R37" V 4145 1200 50  0000 C CNN
-F 1 "56" V 4236 1200 50  0000 C CNN
-F 2 "Resistor_THT:R_Axial_DIN0207_L6.3mm_D2.5mm_P10.16mm_Horizontal" V 4390 1190 50  0001 C CNN
-F 3 "~" H 4350 1200 50  0001 C CNN
-	1    4350 1200
-	0    1    1    0
-$EndComp
 Wire Wire Line
 	3900 1350 3900 1200
@@
 F 0 "R38" V 4895 1850 50  0000 C CNN
 F 1 "567" V 4986 1850 50  0000 C CNN
-F 2 "Resistor_SMD:R_0805_2012Metric_Pad1.15x1.40mm_HandSolder" V 5140 1840 50  0001 C CNN
+F 2 "Resistor_THT:R_Axial_DIN0207_L6.3mm_D2.5mm_P10.16mm_Horizontal" V 5140 1840 50  0001 C CNN
 F 3 "~" H 5100 1850 50  0001 C CNN
 	1    5100 1850
@@
 F 0 "J20" H 15413 2815 50  0000 L CNN
 F 1 "Tensão de Medição" H 15433 1870 50  0000 C CNN
-F 2 "" H 15500 2400 50  0001 C CNN
+F 2 "Connector_PinHeader_2.54mm:PinHeader_1x08_P2.54mm_Vertical" H 15500 2400 50  0001 C CNN
 F 3 "~" H 15500 2400 50  0001 C CNN
 	1    15500 2400
 	1    0    0    1
 $EndComp
+$Comp
+L Device:R_US R37
+U 1 1 5E82D06B
+P 4350 1200
+F 0 "R37" V 4145 1200 50  0000 C CNN
+F 1 "56" V 4236 1200 50  0000 C CNN
+F 2 "Resistor_THT:R_Axial_DIN0207_L6.3mm_D2.5mm_P10.16mm_Horizontal" V 4390 1190 50  0001 C CNN
+F 3 "~" H 4350 1200 50  0001 C CNN
+	1    4350 1200
+	0    1    1    0
+$EndComp
 $EndSCHEMATC

Commit message: Modificação do esquemático e PCB
Parts:
- D1: footprint Diode_SMD:D_SOT-23_ANK -> Diode_THT:D_DO-35_SOD27_P7.62mm_Horizontal
- R38: value 567 -> 75
Changed lines of the file:
@@
 Wire Wire Line
 	7200 1400 7200 2550
+Text Label 14850 2000 0    50   ~ 0
+Vm_out
 Text Label 14850 2200 0    50   ~ 0
-Vm_out
-Text Label 14850 2000 0    50   ~ 0
 Vm_tapOut
 $Comp
@@
 P 5100 1850
 F 0 "R38" V 4895 1850 50  0000 C CNN
-F 1 "567" V 4986 1850 50  0000 C CNN
+F 1 "75" V 4986 1850 50  0000 C CNN
 F 2 "Resistor_THT:R_Axial_DIN0207_L6.3mm_D2.5mm_P10.16mm_Horizontal" V 5140 1840 50  0001 C CNN
 F 3 "~" H 5100 1850 50  0001 C CNN
@@
 F 0 "D1" V 5404 2179 50  0000 L CNN
 F 1 "3,3 V" V 5495 2179 50  0000 L CNN
-F 2 "Diode_SMD:D_SOT-23_ANK" H 5450 2100 50  0001 C CNN
+F 2 "Diode_THT:D_DO-35_SOD27_P7.62mm_Horizontal" H 5450 2100 50  0001 C CNN
 F 3 "~" H 5450 2100 50  0001 C CNN
 	1    5450 2100
@@
 Vm_boost
 Wire Wire Line
+	14850 2200 15300 2200
+Wire Wire Line
 	14850 2000 15300 2000
-Wire Wire Line
-	14850 2200 15300 2200
 Wire Wire Line
 	14750 2400 15300 2400
@@
 Vm_LTSP_25-NP
 $Comp
-L Connector_Generic:Conn_01x08 J20
-U 1 1 5E7D91EF
-P 15500 2400
-F 0 "J20" H 15413 2815 50  0000 L CNN
-F 1 "Tensão de Medição" H 15433 1870 50  0000 C CNN
-F 2 "Connector_PinHeader_2.54mm:PinHeader_1x08_P2.54mm_Vertical" H 15500 2400 50  0001 C CNN
-F 3 "~" H 15500 2400 50  0001 C CNN
-	1    15500 2400
-	1    0    0    1
-$EndComp
-$Comp
 L Device:R_US R37
 U 1 1 5E82D06B
@@
 	0    1    1    0
 $EndComp
+$Comp
+L Connector_Generic:Conn_01x08 J20
+U 1 1 5E7D91EF
+P 15500 2300
+F 0 "J20" H 15413 1772 50  0000 L CNN
+F 1 "Tensão de Medição" H 15433 2715 50  0000 C CNN
+F 2 "Connector_PinHeader_2.54mm:PinHeader_1x08_P2.54mm_Vertical" H 15500 2300 50  0001 C CNN
+F 3 "~" H 15500 2300 50  0001 C CNN
+	1    15500 2300
+	1    0    0    -1
+$EndComp
 $EndSCHEMATC

Commit message: Alteração das labels/Finalização PCB
Parts:
- removed JP7: Jumper_NO_Small, Connector_PinHeader_2.54mm:PinHeader_1x02_P2.54mm_Vertical, symbol Device:Jumper_NO_Small
- renumbered R11 to R10, R12 to R11, R13 to R12, R14 to R13, R15 to R14, R16 to R15, R17 to R16, R18 to R17, R19 to R18, R20 to R19, R21 to R20, R22 to R21, R23 to R22, R24 to R23, R25 to R24, R26 to R25, R27 to R26, R28 to R27, R29 to R28, R30 to R29, R31 to R30, R32 to R31, R33 to R32, R34 to R33, R35 to R34, R36 to R35, R37 to R36, R38 to R37, R5 to R4, R6 to R5, R8 to R6, R9 to R8, R10 to R9, U4 to U3, U3 to U4
Connections:
- net labels removed: +12L
- wire segments 380 -> 378

Commit message: Modificação driver IGBT/LTSP25_NP
Parts:
- removed J10: Comandos PWMs, Connector_PinHeader_2.54mm:PinHeader_1x08_P2.54mm_Vertical, symbol Connector_Generic:Conn_01x08
- removed J15, J16, J17, J18: Driver, Connector_PinHeader_2.54mm:PinHeader_1x07_P2.54mm_Vertical, symbol Connector:Conn_01x07_Female
- removed R30, R31, R32, R33, R34, R35: 340R, Resistor_SMD:R_1206_3216Metric_Pad1.42x1.75mm_HandSolder, symbol Device:R_US
- removed R37: 75, Resistor_THT:R_Axial_DIN0207_L6.3mm_D2.5mm_P10.16mm_Horizontal, symbol Device:R_US
- removed TP10, TP11, TP12, TP13, TP14, TP15, TP16, TP9: TestPoint, Connector_PinHeader_2.54mm:PinHeader_1x01_P2.54mm_Vertical, symbol estabilizador-rescue:TestPoint-Connector
- added C15, C16, C18, C19, C20, C22, C6, C8: 100nF, Capacitor_SMD:C_0805_2012Metric_Pad1.15x1.40mm_HandSolder, symbol Device:C_Small
- added C17, C21: 4.7uF, Capacitor_SMD:CP_Elec_8x10, symbol Device:CP1_Small
- added C7: 100uF, Capacitor_SMD:CP_Elec_8x10, symbol Device:CP1_Small
- added J11, J12: Comandos Boost, Connector_PinHeader_2.54mm:PinHeader_1x04_P2.54mm_Vertical, symbol Connector_Generic:Conn_01x04
- added U5: LM741, symbol Amplifier_Operational:LM741
- added U6, U7: 2ED21814S06J, symbol boost_pfc:2ED21814S06J
- J2: value Alimentação LTSP 25-NP -> Fonte Aux2
- J5: renamed from J9; value Comandos PWMs -> Comandos Inversor
- R28: value 340R -> 6800
- R29: value 340R -> 10000
- R30: renamed from R36; value 56 -> 120; footprint Resistor_THT:R_Axial_DIN0207_L6.3mm_D2.5mm_P10.16mm_Horizontal -> Resistor_SMD:R_1206_3216Metric_Pad1.42x1.75mm_HandSolder
- renumbered C11 to C10, C12 to C11, C13 to C12, C14 to C13, C15 to C14, C6 to C2, C7 to C3, C8 to C4, C9 to C5, C10 to C9, J14 to J10, J20 to J13, J19 to J6, J11 to J7, J12 to J8, J13 to J9
Connections:
- net +12V: no longer R28.1, R29.1
- net +5V: now also C15.2, C18.1, C19.2, C22.1, C6.1, C7.1, C8.2, U5.7 (V+), U6.7 (VCC), U7.7 (VCC)
- net GNDREF: now also R29.1, C15.1, C19.1, C6.2, C7.2, C8.1, J11.2 (Pin_2), J11.4 (Pin_4), J12.2 (Pin_2), J12.4 (Pin_4), U5.4 (V-), U6.3 (VSS), U7.3 (VSS)
- net Gate1: now also U6.12 (HO); no longer J10.1 (Pin_1), TP2.1
- net Gate2: now also U7.12 (HO); no longer J9.1 (Pin_1), TP4.1
- net Gate3: now also U6.6 (LO); no longer J8.1 (Pin_1), TP6.1
- net Gate4: now also U7.6 (LO); no longer J7.1 (Pin_1), TP8.1
- net Gate5: now also J10.1 (Pin_1), TP2.1
- net Gate6: now also J9.1 (Pin_1), TP4.1
- net Gate7: now also J8.1 (Pin_1), TP6.1
- net Gate8: now also J7.1 (Pin_1), TP8.1
- net Source1: now also U4.4 (OUT4), C16.1, C17.2, U6.11 (VS); no longer J10.2 (Pin_2), TP1.1, U4.1 (IN1)
- net Source2: now also C20.1, C21.2, U7.11 (VS); no longer J9.2 (Pin_2), TP3.1
- net Source3: now also C18.2, C22.2, U6.5 (COM), U7.5 (COM); no longer J7.2 (Pin_2), J8.2 (Pin_2), TP5.1, TP7.1
- net Source5: now also J10.2 (Pin_2), TP1.1
- net Source6: now also J9.2 (Pin_2), TP3.1
- net Source7: now also J7.2 (Pin_2), J8.2 (Pin_2), TP5.1, TP7.1
- net Vm_LTSP_25-NP: now also R30.1, U4.8 (Out)
- net at L1.1: now also U4.1 (IN1); no longer U4.4 (OUT4)
- net at U4.7 (Ref): now also R28.2; no longer R30.2
- net PWM8: no longer names the net of R29.2
- net PWM8: now also R28.1, U5.3 (+); no longer R28.2
- new net: R30.2, U5.2 (-), U5.6
- new net: J11.1 (Pin_1), U6.1 (HIN)
- new net: C16.2, C17.1, U6.13 (VB)
- new net: J11.3 (Pin_3), U6.2 (LIN)
- new net: J12.1 (Pin_1), U7.1 (HIN)
- new net: C20.2, C21.1, U7.13 (VB)
- new net: J12.3 (Pin_3), U7.2 (LIN)
Other:
- moved on the sheet: D1, J6, R30, U4

Commit message: Adição dos Testpoints
Parts:
- added TP10, TP11, TP12, TP13, TP14, TP15, TP16, TP9: TestPoint, Connector_PinHeader_2.54mm:PinHeader_1x01_P2.54mm_Vertical, symbol estabilizador-rescue:TestPoint-Connector
Connections:
- net Gate1: now also TP9.1
- net Gate2: now also TP13.1
- net Gate3: now also TP11.1
- net Gate4: now also TP15.1
- net Source1: now also TP10.1
- net Source2: now also TP14.1
- net Source3: now also TP12.1, TP16.1
Changed lines of the file:
@@
 Text Label 10700 8800 2    50   ~ 0
 Source3
-Wire Wire Line
-	10700 8800 10300 8800
 $Comp
 L power:GNDREF #PWR?
@@
 Text Label 13650 8800 2    50   ~ 0
 Source4
-Wire Wire Line
-	13650 8800 13250 8800
 $Comp
 L power:GNDREF #PWR?
@@
 Wire Wire Line
 	13750 7450 13750 7800
-Wire Wire Line
-	10750 8100 11050 8100
-Wire Wire Line
-	10750 8200 11050 8200
-Wire Wire Line
-	13700 8100 14000 8100
-Wire Wire Line
-	13700 8200 14000 8200
 $Comp
 L Device:C_Small C9
@@
 Text Label 11550 7900 2    50   ~ 0
 Source1
-Wire Wire Line
-	11550 7900 11150 7900
 Connection ~ 11150 7900
 Text Label 14500 7900 2    50   ~ 0
 Source2
-Wire Wire Line
-	14500 7900 14100 7900
 Connection ~ 14100 7900
+$Comp
+L estabilizador-rescue:TestPoint-Connector TP9
+U 1 1 5E6A657C
+P 11100 8100
+F 0 "TP9" H 11158 8174 50  0000 L CNN
+F 1 "TestPoint" H 11158 8129 50  0001 L CNN
+F 2 "Connector_PinHeader_2.54mm:PinHeader_1x01_P2.54mm_Vertical" H 11300 8100 50  0001 C CNN
+F 3 "~" H 11300 8100 50  0001 C CNN
+	1    11100 8100
+	1    0    0    -1
+$EndComp
+$Comp
+L estabilizador-rescue:TestPoint-Connector TP11
+U 1 1 5E6CE798
+P 11100 8200
+F 0 "TP11" H 10866 8274 50  0000 L CNN
+F 1 "TestPoint" H 11158 8229 50  0001 L CNN
+F 2 "Connector_PinHeader_2.54mm:PinHeader_1x01_P2.54mm_Vertical" H 11300 8200 50  0001 C CNN
+F 3 "~" H 11300 8200 50  0001 C CNN
+	1    11100 8200
+	-1   0    0    1
+$EndComp
+$Comp
+L estabilizador-rescue:TestPoint-Connector TP10
+U 1 1 5E6F7281
+P 11600 7900
+F 0 "TP10" H 11658 7974 50  0000 L CNN
+F 1 "TestPoint" H 11658 7929 50  0001 L CNN
+F 2 "Connector_PinHeader_2.54mm:PinHeader_1x01_P2.54mm_Vertical" H 11800 7900 50  0001 C CNN
+F 3 "~" H 11800 7900 50  0001 C CNN
+	1    11600 7900
+	1    0    0    -1
+$EndComp
+$Comp
+L estabilizador-rescue:TestPoint-Connector TP12
+U 1 1 5E7477E4
+P 10750 8800
+F 0 "TP12" H 10808 8874 50  0000 L CNN
+F 1 "TestPoint" H 10808 8829 50  0001 L CNN
+F 2 "Connector_PinHeader_2.54mm:PinHeader_1x01_P2.54mm_Vertical" H 10950 8800 50  0001 C CNN
+F 3 "~" H 10950 8800 50  0001 C CNN
+	1    10750 8800
+	1    0    0    -1
+$EndComp
+$Comp
+L estabilizador-rescue:TestPoint-Connector TP13
+U 1 1 5E76F53B
+P 14050 8100
+F 0 "TP13" H 14108 8174 50  0000 L CNN
+F 1 "TestPoint" H 14108 8129 50  0001 L CNN
+F 2 "Connector_PinHeader_2.54mm:PinHeader_1x01_P2.54mm_Vertical" H 14250 8100 50  0001 C CNN
+F 3 "~" H 14250 8100 50  0001 C CNN
+	1    14050 8100
+	1    0    0    -1
+$EndComp
+$Comp
+L estabilizador-rescue:TestPoint-Connector TP14
+U 1 1 5E7BF769
+P 14550 7900
+F 0 "TP14" H 14608 7974 50  0000 L CNN
+F 1 "TestPoint" H 14608 7929 50  0001 L CNN
+F 2 "Connector_PinHeader_2.54mm:PinHeader_1x01_P2.54mm_Vertical" H 14750 7900 50  0001 C CNN
+F 3 "~" H 14750 7900 50  0001 C CNN
+	1    14550 7900
+	1    0    0    -1
+$EndComp
+$Comp
+L estabilizador-rescue:TestPoint-Connector TP16
+U 1 1 5E7E7515
+P 13700 8800
+F 0 "TP16" H 13758 8874 50  0000 L CNN
+F 1 "TestPoint" H 13758 8829 50  0001 L CNN
+F 2 "Connector_PinHeader_2.54mm:PinHeader_1x01_P2.54mm_Vertical" H 13900 8800 50  0001 C CNN
+F 3 "~" H 13900 8800 50  0001 C CNN
+	1    13700 8800
+	1    0    0    -1
+$EndComp
+Wire Wire Line
+	10750 8100 11100 8100
+Wire Wire Line
+	10750 8200 11100 8200
+Wire Wire Line
+	11150 7900 11600 7900
+Wire Wire Line
+	10300 8800 10750 8800
+Wire Wire Line
+	14100 7900 14550 7900
+Wire Wire Line
+	13700 8100 14050 8100
+Wire Wire Line
+	13700 8200 14050 8200
+Wire Wire Line
+	13250 8800 13700 8800
+$Comp
+L estabilizador-rescue:TestPoint-Connector TP15
+U 1 1 5E79751A
+P 14050 8200
+F 0 "TP15" H 13858 8274 50  0000 L CNN
+F 1 "TestPoint" H 14108 8229 50  0001 L CNN
+F 2 "Connector_PinHeader_2.54mm:PinHeader_1x01_P2.54mm_Vertical" H 14250 8200 50  0001 C CNN
+F 3 "~" H 14250 8200 50  0001 C CNN
+	1    14050 8200
+	-1   0    0    1
+$EndComp
 $EndSCHEMATC

Commit message: Modificação drivers e chaves
Parts:
- removed C15, C16, C18, C19, C20, C22, C6: 100nF, Capacitor_SMD:C_0805_2012Metric_Pad1.15x1.40mm_HandSolder, symbol Device:C_Small
- removed C17, C21: 4.7uF, Capacitor_SMD:CP_Elec_8x10, symbol Device:CP1_Small
- removed J11, J12: Comandos Boost, Connector_PinHeader_2.54mm:PinHeader_1x04_P2.54mm_Vertical, symbol Connector_Generic:Conn_01x04
- removed Q1, Q2, Q3, Q4: IRG4PF50W, Package_TO_SOT_THT:TO-247-3_Vertical, symbol Transistor_IGBT:IRG4PF50W
- removed R10, R11, R14, R15: 10K, Resistor_THT:R_Axial_DIN0414_L11.9mm_D4.5mm_P15.24mm_Horizontal, symbol Device:R_US
- removed R18: 10K, Resistor_THT:R_Axial_DIN0207_L6.3mm_D2.5mm_P10.16mm_Horizontal, symbol Device:R_US
- removed U5: LM741, symbol Amplifier_Operational:LM741
- removed U6, U7: 2ED21814S06J, symbol boost_pfc:2ED21814S06J
- added C1: 4700uF, Capacitor_THT:CP_Radial_D18.0mm_P7.50mm, symbol Device:CP1_Small
- added C3: 910nF, Capacitor_THT:C_Rect_L29.0mm_W7.6mm_P27.50mm_MKT, symbol Device:C_Small
- added J11: Comandos Inversor, Connector_PinHeader_2.54mm:PinHeader_1x08_P2.54mm_Vertical, symbol Connector_Generic:Conn_01x08
- added J12, J13, J14, J15: Driver, Connector_PinHeader_2.54mm:PinHeader_1x07_P2.54mm_Vertical, symbol Connector:Conn_01x07_Female
- added Q1, Q2, Q3, Q4: IRF540N, boost_pfc:TO-220-3 Heatsink, symbol Transistor_FET:IRF540N
- added R23, R24, R25, R26, R27, R28, R29, R30: 340R, Resistor_SMD:R_1206_3216Metric_Pad1.42x1.75mm_HandSolder, symbol Device:R_US
- C2: renamed from C1; value 2700uF -> 4700uF
- C4: renamed from C5; value 690nF -> 910nF
- C5: renamed from C4; value 690nF -> 910nF
- C6: renamed from C2; value 390nF -> 750nF
- C7: renamed from C3; value 390nF -> 750nF
- J5: value Comandos Inversor -> Comandos Boost
- L2: footprint boost_pfc:NEE_45-45 -> boost_pfc:NEE_42-20
- R10: renamed from R12; value 10k -> 5k6; footprint Resistor_THT:R_Axial_DIN0414_L11.9mm_D4.5mm_P15.24mm_Horizontal -> Resistor_THT:R_Axial_DIN0411_L9.9mm_D3.6mm_P15.24mm_Horizontal
- R11: renamed from R13; value 2K2 -> 5k6; footprint Resistor_THT:R_Axial_DIN0414_L11.9mm_D4.5mm_P15.24mm_Horizontal -> Resistor_THT:R_Axial_DIN0411_L9.9mm_D3.6mm_P15.24mm_Horizontal
- R12: renamed from R16; value 10K -> 5k6; footprint Resistor_THT:R_Axial_DIN0414_L11.9mm_D4.5mm_P15.24mm_Horizontal -> Resistor_THT:R_Axial_DIN0411_L9.9mm_D3.6mm_P15.24mm_Horizontal
- R13: renamed from R17; value 10K -> 5k6; footprint Resistor_THT:R_Axial_DIN0414_L11.9mm_D4.5mm_P15.24mm_Horizontal -> Resistor_THT:R_Axial_DIN0411_L9.9mm_D3.6mm_P15.24mm_Horizontal
- R14: renamed from R19; value 10K -> 1k5; footprint Resistor_THT:R_Axial_DIN0207_L6.3mm_D2.5mm_P10.16mm_Horizontal -> Resistor_THT:R_Axial_DIN0309_L9.0mm_D3.2mm_P12.70mm_Horizontal
- R31: renamed from R30; value 120 -> 200
- R32: renamed from R28; value 6800 -> 10k
- R33: renamed from R29; value 10000 -> 15k
- R9: value 3K3 -> 750; footprint Resistor_THT:R_Axial_DIN0309_L9.0mm_D3.2mm_P12.70mm_Horizontal -> Resistor_THT:R_Axial_DIN0207_L6.3mm_D2.5mm_P10.16mm_Horizontal
- renumbered C9 to C10, C10 to C11, C11 to C12, C12 to C13, C13 to C14, C14 to C15, C7 to C8, C8 to C9, J5 to J16, J6 to J17, J7 to J18, J8 to J19, J13 to J20, R20 to R15, R21 to R16, R22 to R17, R23 to R18, R24 to R19, R25 to R20, R26 to R21, R27 to R22
Connections:
- net -12V: no longer J6.3 (Pin_3), U1.6 (V-), U2.6 (V-), U3.6 (V-)
- net GNDREF: now also J11.2 (Pin_2), J11.4 (Pin_4), J11.6 (Pin_6), J11.8 (Pin_8), J12.4 (Pin_4), J12.7 (Pin_7), J13.4 (Pin_4), J13.7 (Pin_7), J14.4 (Pin_4), J14.7 (Pin_7), J15.4 (Pin_4), J15.7 (Pin_7)
- net Gate1: now also J10.1 (Pin_1), TP2.1, Q1.1 (G); no longer TP9.1
- net Gate2: now also J9.1 (Pin_1), TP4.1, Q2.1 (G); no longer TP13.1
- net Gate3: now also J8.1 (Pin_1), TP6.1, Q3.1 (G); no longer TP11.1
- net Gate4: now also J7.1 (Pin_1), TP8.1, Q4.1 (G); no longer TP15.1
- net Gate5: now also TP10.1, J15.1 (Pin_1); no longer J10.1 (Pin_1), TP2.1
- net Gate6: now also TP12.1, J14.1 (Pin_1); no longer J9.1 (Pin_1), TP4.1
- net Gate7: now also TP14.1, J13.1 (Pin_1); no longer J8.1 (Pin_1), TP6.1
- net Gate8: now also TP16.1, J12.1 (Pin_1); no longer J7.1 (Pin_1), TP8.1
- net Source1: now also J10.2 (Pin_2), TP1.1, Q1.3 (S), Q3.2 (D); no longer TP10.1
- net Source2: now also J9.2 (Pin_2), TP3.1, Q2.3 (S), Q4.2 (D); no longer TP14.1
- net Source3: now also J7.2 (Pin_2), J8.2 (Pin_2), TP5.1, TP7.1, C1.2, Q3.3 (S), Q4.3 (S); no longer TP12.1, TP16.1
- net Source5: now also TP9.1, J15.2 (Pin_2); no longer J10.2 (Pin_2), TP1.1
- net Source6: now also R10.2, TP11.1, C3.2, J14.2 (Pin_2); no longer J9.2 (Pin_2), TP3.1
- net Source7: now also TP13.1, TP15.1, J12.2 (Pin_2), J13.2 (Pin_2); no longer J7.2 (Pin_2), J8.2 (Pin_2), TP5.1, TP7.1
- net Vboost+: now also R14.2, C1.1, Q1.2 (D), Q2.2 (D)
- net Vm_LTSP_25-NP: now also R32.1, R33.2; no longer R31.1, U4.8 (Out)
- net VtapOut: now also R12.2
- net at C4.1, C5.1, JP3.1 (A): now also C3.1
- net at U4.7 (Ref): now also R31.2; no longer R32.2
- net +12V renamed +15V
- net +15V: now also J12.5 (Pin_5), J13.5 (Pin_5), J14.5 (Pin_5), J15.5 (Pin_5), R23.1, R24.1, R25.1, R26.1, R27.1, R28.1, R29.1, R30.1
- new net: R31.1, R32.2, U4.8 (Out)
- new net -15V: J6.3 (Pin_3), U1.6 (V-), U2.6 (V-), U3.6 (V-)
- new net PWM5: J11.1 (Pin_1), J15.6 (Pin_6), R29.2, R30.2
- new net PWM6: J11.3 (Pin_3), J14.6 (Pin_6), R27.2, R28.2
- new net PWM7: J11.5 (Pin_5), J13.6 (Pin_6), R25.2, R26.2
- new net PWM8: J11.7 (Pin_7), J12.6 (Pin_6), R23.2, R24.2
Other:
- moved on the sheet: C2, D1, J10, J17, J19, J5, J6, J7, J8, J9, R15, R16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
