File: estabilizador.kicad_pcb (KiCad board)
At the start: 2 copper layers, 259.7 x 125.1 mm, 91 parts, among them J1 Tensão de Entrada, J10 Driver, J11 Tensão do Estágio de Reles, J12 Tensão do Estágio do Inversor, J13 Tensão de Saída Total, J14 Tensão de Medição, J15 Tap AUX2, J2 Autotransformador, J3 Comandos Reles, J4 Tap AUX1, J5 Comandos PWMs, J6 Fonte Aux, J7 Driver, J8 Driver, J9 Driver, K1 RT42xxxx, K2 RT42xxxx, K3 RT42xxxx, Q1 BC517, Q2 BC517, Q3 IRF840N, Q4 IRF840N, Q5 BC517, Q6 IRF840N, Q7 IRF840N, U1 LV20-P, U2 LV25-P

Commit message: v2
Parts:
- removed C2, C3: 1000uF, Capacitor_THT:CP_Radial_D18.0mm_P7.50mm
- removed C4: 390nF, Capacitor_THT:C_Rect_L26.5mm_W7.0mm_P22.50mm_MKS4
- removed C5: 690nF, Capacitor_THT:C_Rect_L29.0mm_W7.6mm_P27.50mm_MKT
- removed D2, D3, D4: 1N4148, Diode_THT:D_DO-35_SOD27_P7.62mm_Horizontal
- removed JP7, JP8, JP9: Jumper_NO_Small, Connector_PinHeader_2.54mm:PinHeader_1x02_P2.54mm_Vertical
- removed K1: RT42xxxx, Relay:Relay_DPDT_model_A
- removed K2, K3: RT42xxxx, Relay:Relay_DPDT_model_B
- added J16: Driver, Connector_PinHeader_2.54mm:PinHeader_1x07_P2.54mm_Vertical, F.Cu at (90.8, 138.4)
- added J17: Driver, Connector_PinHeader_2.54mm:PinHeader_1x07_P2.54mm_Vertical, F.Cu at (67.9, 138.4)
- added J18: Driver, Connector_PinHeader_2.54mm:PinHeader_1x07_P2.54mm_Vertical, F.Cu at (45.1, 138.4)
- added J19: Fonte Aux, Connector_PinHeader_2.54mm:PinHeader_1x03_P2.54mm_Vertical, F.Cu at (53.3, 156.2)
- added J20: Tensão de Medição, Connector_PinHeader_2.54mm:PinHeader_1x08_P2.54mm_Vertical, F.Cu at (181.0, 156.2)
- added L2: L_Core_Ferrite, boost_pfc:NEE_45-45, F.Cu at (53.3, 104.1)
- added Q8: IRF840N, boost_pfc:TO-220-3 Heatsink, F.Cu at (113.7, 126.4)
- added R28: 340R, Resistor_SMD:R_1206_3216Metric_Pad1.42x1.75mm_HandSolder, B.Cu at (125.1, 142.2)
- added R29: 340R, Resistor_SMD:R_1206_3216Metric_Pad1.42x1.75mm_HandSolder, B.Cu at (125.1, 145.4)
- added R30: 340R, Resistor_SMD:R_1206_3216Metric_Pad1.42x1.75mm_HandSolder, B.Cu at (102.2, 145.4)
- added R31: 340R, Resistor_SMD:R_1206_3216Metric_Pad1.42x1.75mm_HandSolder, B.Cu at (102.2, 142.2)
- added R32: 340R, Resistor_SMD:R_1206_3216Metric_Pad1.42x1.75mm_HandSolder, B.Cu at (79.4, 142.2)
- added R33: 340R, Resistor_SMD:R_1206_3216Metric_Pad1.42x1.75mm_HandSolder, B.Cu at (79.4, 145.4)
- added R34: 340R, Resistor_SMD:R_1206_3216Metric_Pad1.42x1.75mm_HandSolder, B.Cu at (56.5, 145.4)
- added R35: 340R, Resistor_SMD:R_1206_3216Metric_Pad1.42x1.75mm_HandSolder, B.Cu at (56.5, 142.2)
- added R36: 56, Resistor_THT:R_Axial_DIN0207_L6.3mm_D2.5mm_P10.16mm_Horizontal, F.Cu at (271.1, 104.8)
- added R37: 75, Resistor_THT:R_Axial_DIN0207_L6.3mm_D2.5mm_P10.16mm_Horizontal, F.Cu at (239.4, 104.8)
- added TP10: TestPoint, Connector_PinHeader_2.54mm:PinHeader_1x01_P2.54mm_Vertical, F.Cu at (43.8, 144.1)
- added TP11: TestPoint, Connector_PinHeader_2.54mm:PinHeader_1x01_P2.54mm_Vertical, F.Cu at (70.5, 144.1)
- added TP12: TestPoint, Connector_PinHeader_2.54mm:PinHeader_1x01_P2.54mm_Vertical, F.Cu at (66.7, 144.1)
- added TP13: TestPoint, Connector_PinHeader_2.54mm:PinHeader_1x01_P2.54mm_Vertical, F.Cu at (93.3, 144.1)
- added TP14: TestPoint, Connector_PinHeader_2.54mm:PinHeader_1x01_P2.54mm_Vertical, F.Cu at (89.5, 144.1)
- added TP15: TestPoint, Connector_PinHeader_2.54mm:PinHeader_1x01_P2.54mm_Vertical, F.Cu at (116.2, 144.1)
- added TP16: TestPoint, Connector_PinHeader_2.54mm:PinHeader_1x01_P2.54mm_Vertical, F.Cu at (112.4, 144.1)
- added TP9: TestPoint, Connector_PinHeader_2.54mm:PinHeader_1x01_P2.54mm_Vertical, F.Cu at (47.6, 144.1)
- added U3: LV25-P, Sensor_Voltage:LEM_LV25-P, F.Cu at (220.3, 107.3)
- added U4: LTSP_25-NP, Sensor_Current:LEM_LTSR-NP, F.Cu at (251.8, 90.8)
- C1: value 1000uF -> 2700uF
- C12: value 2uF -> 100nF; footprint Capacitor_THT:C_Rect_L29.0mm_W7.6mm_P27.50mm_MKT -> Capacitor_SMD:C_0805_2012Metric_Pad1.15x1.40mm_HandSolder; moved to B.Cu
- C13: value 2uF -> 100uF; footprint Capacitor_THT:C_Rect_L29.0mm_W7.6mm_P27.50mm_MKT -> Capacitor_SMD:CP_Elec_8x10; moved to B.Cu
- C14: value 1uF -> 100nF; footprint Capacitor_THT:C_Rect_L29.0mm_W7.6mm_P27.50mm_MKT -> Capacitor_SMD:C_0805_2012Metric_Pad1.15x1.40mm_HandSolder; moved to B.Cu
- C15: value 1uF -> 100uF; footprint Capacitor_THT:C_Rect_L29.0mm_W7.6mm_P27.50mm_MKT -> Capacitor_SMD:CP_Elec_8x10; moved to B.Cu
- C6: value 690nF -> 390nF; footprint Capacitor_THT:C_Rect_L29.0mm_W7.6mm_P27.50mm_MKT -> Capacitor_THT:C_Rect_L26.5mm_W7.0mm_P22.50mm_MKS4
- C8: value 100nF -> 690nF; footprint Capacitor_SMD:C_0805_2012Metric_Pad1.15x1.40mm_HandSolder -> Capacitor_THT:C_Rect_L29.0mm_W7.6mm_P27.50mm_MKT; moved to F.Cu
- C9: value 100uF -> 690nF; footprint Capacitor_SMD:CP_Elec_8x10 -> Capacitor_THT:C_Rect_L29.0mm_W7.6mm_P27.50mm_MKT; moved to F.Cu
- D1: value GBU8J -> 3,3 V; footprint Diode_THT:Diode_Bridge_Vishay_KBU -> Diode_THT:D_DO-35_SOD27_P7.62mm_Horizontal
- J10, J9: value Driver -> Comandos PWMs; footprint Connector_PinHeader_2.54mm:PinHeader_1x07_P2.54mm_Vertical -> Connector_PinHeader_2.54mm:PinHeader_1x08_P2.54mm_Vertical
- J11: value Tensão do Estágio de Reles -> Driver; footprint Connector_Phoenix_MSTB:PhoenixContact_MSTBVA_2,5_2-G-5,08_1x02_P5.08mm_Vertical -> Connector_PinHeader_2.54mm:PinHeader_1x07_P2.54mm_Vertical
- J12: value Tensão do Estágio do Inversor -> Driver; footprint Connector_Phoenix_MSTB:PhoenixContact_MSTBVA_2,5_2-G-5,08_1x02_P5.08mm_Vertical -> Connector_PinHeader_2.54mm:PinHeader_1x07_P2.54mm_Vertical
- J13: value Tensão de Saída Total -> Driver; footprint Connector_Phoenix_MSTB:PhoenixContact_MSTBVA_2,5_2-G-5,08_1x02_P5.08mm_Vertical -> Connector_PinHeader_2.54mm:PinHeader_1x07_P2.54mm_Vertical
- J14: value Tensão de Medição -> Driver; footprint Connector_PinHeader_2.54mm:PinHeader_1x04_P2.54mm_Vertical -> Connector_PinHeader_2.54mm:PinHeader_1x07_P2.54mm_Vertical
- J15: value Tap AUX2 -> Driver; footprint Connector_Phoenix_MSTB:PhoenixContact_MSTBVA_2,5_4-G-5,08_1x04_P5.08mm_Vertical -> Connector_PinHeader_2.54mm:PinHeader_1x07_P2.54mm_Vertical
- J2: value Autotransformador -> Alimentação LTSP 25-NP; footprint Connector_Phoenix_MSTB:PhoenixContact_MSTBVA_2,5_5-G-5,08_1x05_P5.08mm_Vertical -> Connector_PinHeader_2.54mm:PinHeader_1x02_P2.54mm_Vertical
- J3: value Comandos Reles -> Tap AUX1; footprint Connector_PinHeader_2.54mm:PinHeader_1x06_P2.54mm_Vertical -> Connector_Phoenix_MSTB:PhoenixContact_MSTBVA_2,5_2-G-5,08_1x02_P5.08mm_Vertical
- J4: value Tap AUX1 -> Screw_Terminal_01x02
- J5: value Comandos PWMs -> Tensão do Estabilizador; footprint Connector_PinHeader_2.54mm:PinHeader_1x08_P2.54mm_Vertical -> Connector_Phoenix_MSTB:PhoenixContact_MSTBVA_2,5_2-G-5,08_1x02_P5.08mm_Vertical
- J6: value Fonte Aux -> Tensão do Estágio do Inversor; footprint Connector_PinHeader_2.54mm:PinHeader_1x03_P2.54mm_Vertical -> Connector_Phoenix_MSTB:PhoenixContact_MSTBVA_2,5_2-G-5,08_1x02_P5.08mm_Vertical
- J7: value Driver -> Tensão de Saída Total; footprint Connector_PinHeader_2.54mm:PinHeader_1x07_P2.54mm_Vertical -> Connector_Phoenix_MSTB:PhoenixContact_MSTBVA_2,5_2-G-5,08_1x02_P5.08mm_Vertical
- J8: value Driver -> Tensão de Saída do Boost; footprint Connector_PinHeader_2.54mm:PinHeader_1x07_P2.54mm_Vertical -> Connector_Phoenix_MSTB:PhoenixContact_MSTBVA_2,5_2-G-5,08_1x02_P5.08mm_Vertical
- JP3: value Jumper_NO_Small -> Jumper_3_Bridged12; footprint Connector_PinHeader_2.54mm:PinHeader_1x02_P2.54mm_Vertical -> Connector_PinHeader_2.54mm:PinHeader_1x03_P2.54mm_Vertical
- JP4: value Jumper_3_Bridged12 -> Jumper_NO_Small; footprint Connector_PinHeader_2.54mm:PinHeader_1x03_P2.54mm_Vertical -> Connector_PinHeader_2.54mm:PinHeader_1x02_P2.54mm_Vertical
- L1: footprint Inductors:Inductor_EE4220 -> boost_pfc:NEE_30-14
- Q1, Q2: value BC517 -> IRG4PF50W; footprint Package_TO_SOT_THT:TO-92_Inline_Wide -> Package_TO_SOT_THT:TO-247-3_Vertical
- Q3, Q4: value IRF840N -> IRG4PF50W; footprint transistors:TO-220-3 Heatsink -> Package_TO_SOT_THT:TO-247-3_Vertical
- Q5: value BC517 -> IRF840N; footprint Package_TO_SOT_THT:TO-92_Inline_Wide -> boost_pfc:TO-220-3 Heatsink
- Q6, Q7: footprint transistors:TO-220-3 Heatsink -> boost_pfc:TO-220-3 Heatsink
- R1, R3, R5: value 100K -> 10k
- R11: value 3K3 -> 10K; footprint Resistor_THT:R_Axial_DIN0309_L9.0mm_D3.2mm_P12.70mm_Horizontal -> Resistor_THT:R_Axial_DIN0414_L11.9mm_D4.5mm_P15.24mm_Horizontal
- R12: value 10K -> 10k
- R13: value 10k -> 2K2
- R14, R15, R16: value 10k -> 10K
- R17: value 340R -> 10K; footprint Resistor_SMD:R_1206_3216Metric_Pad1.42x1.75mm_HandSolder -> Resistor_THT:R_Axial_DIN0414_L11.9mm_D4.5mm_P15.24mm_Horizontal; moved to F.Cu
- R18, R19: value 340R -> 10K; footprint Resistor_SMD:R_1206_3216Metric_Pad1.42x1.75mm_HandSolder -> Resistor_THT:R_Axial_DIN0207_L6.3mm_D2.5mm_P10.16mm_Horizontal; moved to F.Cu
- R2, R4, R6, R7: value 340R -> 10k; footprint Resistor_SMD:R_1206_3216Metric_Pad1.42x1.75mm_HandSolder -> Resistor_SMD:R_0805_2012Metric_Pad1.15x1.40mm_HandSolder
- R21, R22, R23: value 10K -> 340R; footprint Resistor_SMD:R_0805_2012Metric_Pad1.15x1.40mm_HandSolder -> Resistor_SMD:R_1206_3216Metric_Pad1.42x1.75mm_HandSolder
- R24, R25, R26, R27: value 10k -> 340R; footprint Resistor_SMD:R_0805_2012Metric_Pad1.15x1.40mm_HandSolder -> Resistor_SMD:R_1206_3216Metric_Pad1.42x1.75mm_HandSolder
- R8: value 10K -> 10k; footprint Resistor_THT:R_Axial_DIN0414_L11.9mm_D4.5mm_P15.24mm_Horizontal -> Resistor_SMD:R_0805_2012Metric_Pad1.15x1.40mm_HandSolder; moved to B.Cu
- R9: value 10K -> 3K3; footprint Resistor_THT:R_Axial_DIN0414_L11.9mm_D4.5mm_P15.24mm_Horizontal -> Resistor_THT:R_Axial_DIN0309_L9.0mm_D3.2mm_P12.70mm_Horizontal
- moved TP7 279.0 mm to (315.0, 144.1), turned to 180 degrees
- moved TP8 279.0 mm to (311.1, 144.1), turned to 180 degrees
- moved R20 278.9 mm to (323.9, 142.2)
- moved Q3 256.3 mm to (289.6, 124.5)
- moved J13 252.1 mm to (266.7, 138.4)
- moved R24 244.6 mm to (278.1, 142.2)
- moved Q4 233.4 mm to (312.4, 124.5)
- moved TP5 233.3 mm to (292.1, 144.1), turned to 180 degrees
- moved TP6 233.3 mm to (288.3, 144.1), turned to 180 degrees
- moved R4 222.9 mm to (313.7, 130.2)
- moved J9 222.0 mm to (276.9, 156.2)
- moved L1 221.9 mm to (283.8, 62.2), turned to 0 degrees
- moved J2 214.8 mm to (69.8, 156.2), turned to 90 degrees
- moved R25 199.6 mm to (278.1, 145.4)
- moved R26 199.2 mm to (255.3, 142.4)
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Connections:
- C1 pad 1: /HI_in_inv -> /Vboost+
- C1 pad 2: /LO_in_inv -> /Source3
- C12 pad 1: Net-(C12-Pad1) -> -12V
- C12 pad 2: Net-(C12-Pad2) -> +12V
- C13 pad 1: /Source3 -> +12V
- C13 pad 2: /Source4 -> -12V
- C14 pad 1: Net-(C12-Pad2) -> -12V
- C14 pad 2: /Source3 -> +12V
- C15 pad 1: Net-(C12-Pad1) -> +12V
- C15 pad 2: /Source4 -> -12V
- C6 pad 1: Net-(C5-Pad1) -> Net-(C6-Pad1)
- C6 pad 2: /Source2 -> Net-(C6-Pad2)
- C7 pad 1: Net-(C4-Pad2) -> Net-(C6-Pad2)
- C7 pad 2: /Source2 -> /Source6
- C8 pad 1: -12V -> Net-(C8-Pad1)
- C8 pad 2: +12V -> /Source6
- C9 pad 1: +12V -> Net-(C8-Pad1)
- C9 pad 2: -12V -> /Source6
- D1 pad 1: /HI_in_inv -> /Vm_LTSP_25-NP
- D1 pad 2: /VauxA -> GNDREF
- J1 pad 2: LINE -> /VtapOut
- J10 pad 1: /Gate1 -> /PWM5
- J10 pad 2: /Source1 -> GNDREF
- J10 pad 3: Net-(J10-Pad3) -> /PWM6
- J10 pad 5: +12V -> /PWM7
- J10 pad 6: /PWM1 -> GNDREF
- J10 pad 7: GNDREF -> /PWM8
- J11 pad 1: NEUT -> /Gate4
- J11 pad 2: /VtapOut -> /Source3
- J12 pad 1: /Vinv- -> /Gate3
- J12 pad 2: /Source2 -> /Source3
- J13 pad 1: /Source2 -> /Gate2
- J13 pad 2: NEUT -> /Source2
- J14 pad 1: GNDREF -> /Gate1
- J14 pad 2: /Vm_out -> /Source1
- J14 pad 3: GNDREF -> Net-(J14-Pad3)
- J14 pad 4: /Vm_in -> GNDREF
- J15 pad 1: Net-(C12-Pad1) -> /Gate8
- J15 pad 2: Net-(C12-Pad2) -> /Source7
- J15 pad 3: /Source3 -> Net-(J15-Pad3)
- J15 pad 4: /Source4 -> GNDREF
- J2 pad 1: /Vtap1 -> +5V
- J2 pad 2: /VtapIn -> GNDREF
- J3 pad 1: /RL1 -> /VauxA
- J3 pad 2: GNDREF -> /Source2
- J4 pad 1: /VauxA -> Net-(J4-Pad1)
- J4 pad 2: /VauxB -> /Source7
- J5 pad 1: /PWM1 -> NEUT
- J5 pad 2: GNDREF -> /VtapOut
- J6 pad 1: +12V -> /Vinv-
- J6 pad 2: GNDREF -> /Source6
- J7 pad 1: /Gate4 -> /Source6
- J7 pad 2: /Source4 -> NEUT
- J8 pad 1: /Gate3 -> /Vboost+
- J9 pad 1: /Gate2 -> /PWM1
- J9 pad 2: /Source2 -> GNDREF
- J9 pad 3: Net-(J9-Pad3) -> /PWM2
- J9 pad 5: +12V -> /PWM3
- J9 pad 6: /PWM2 -> GNDREF
- J9 pad 7: GNDREF -> /PWM4
- JP1 pad 1: Net-(C12-Pad2) -> Net-(J4-Pad1)
- JP1 pad 2: /HI_in_inv -> /Vboost+
- JP2 pad 1: /Source3 -> /Source7
- JP2 pad 2: /LO_in_inv -> /Source3
- JP3 pad 1: /VtapOut -> Net-(C8-Pad1)
- JP4 pad 1: Net-(C5-Pad1) -> /VtapOut
- JP6 pad 3: /Source2 -> /Source6
- L1 pad 1: /Source1 -> Net-(L1-Pad1)
- L1 pad 2: /Vinv- -> /VauxA
- Q1 pad 1: Net-(D2-Pad2) -> /Gate1
- Q1 pad 2: Net-(Q1-Pad2) -> /Vboost+
- Q1 pad 3: GNDREF -> /Source1
- Q2 pad 1: Net-(D3-Pad2) -> /Gate2
- Q2 pad 2: Net-(Q2-Pad2) -> /Vboost+
- Q2 pad 3: GNDREF -> /Source2
- Q3 pad 1: /Gate1 -> /Gate3
- Q3 pad 2: Net-(C12-Pad2) -> /Source1
- Q3 pad 3: /Source1 -> /Source3
- Q4 pad 1: /Gate3 -> /Gate4
- Q4 pad 2: /Source1 -> /Source2
- Q5 pad 1: Net-(D4-Pad2) -> /Gate5
- Q5 pad 2: Net-(Q5-Pad2) -> Net-(J4-Pad1)
- Q5 pad 3: GNDREF -> /Source5
- Q6 pad 1: /Gate2 -> /Gate6
- Q6 pad 2: Net-(C12-Pad1) -> Net-(J4-Pad1)
- Q6 pad 3: /Source2 -> /Source6
- Q7 pad 1: /Gate4 -> /Gate7
- Q7 pad 2: /Source2 -> /Source5
- Q7 pad 3: /Source4 -> /Source7
- R1 pad 1: Net-(Q1-Pad2) -> /Gate1
- R1 pad 2: /RL1 -> /Source1
- R10 pad 2: Net-(R10-Pad2) -> /Source6
- R11 pad 1: Net-(JP5-Pad3) -> Net-(R11-Pad1)
- R11 pad 2: /Vinv- -> Net-(R10-Pad1)
- R12 pad 2: Net-(R12-Pad2) -> Net-(R11-Pad1)
- R13 pad 1: Net-(R13-Pad1) -> Net-(JP5-Pad1)
- R13 pad 2: Net-(R10-Pad1) -> Net-(R12-Pad1)
- R14 pad 2: Net-(R12-Pad1) -> /VtapOut
- R15 pad 1: Net-(JP5-Pad1) -> Net-(R15-Pad1)
- R15 pad 2: Net-(R13-Pad1) -> Net-(R14-Pad1)
- R16 pad 2: Net-(R14-Pad1) -> Net-(R15-Pad1)
- R17 pad 1: +12V -> Net-(R17-Pad1)
- R17 pad 2: /PWM4 -> Net-(R16-Pad1)
- R18 pad 1: +12V -> Net-(R18-Pad1)
- R18 pad 2: /PWM3 -> /Vboost+
- R19 pad 1: +12V -> Net-(R19-Pad1)
- R19 pad 2: /PWM2 -> Net-(R18-Pad1)
- R2 pad 1: +12V -> /Gate2
- R2 pad 2: /PWM4 -> /Source2
- R20 pad 2: /PWM1 -> /PWM4
- R21 pad 1: /RL1 -> +12V
- R21 pad 2: +12L -> /PWM4
- R22 pad 1: /RL2 -> +12V
- R22 pad 2: +12L -> /PWM3
- R23 pad 1: /RL3 -> +12V
- R23 pad 2: +12L -> /PWM3
- R24 pad 1: /Gate1 -> +12V
- R24 pad 2: /Source1 -> /PWM2
- R25 pad 1: /Gate3 -> +12V
- R25 pad 2: /Source3 -> /PWM2
- R26 pad 1: /Gate2 -> +12V
- R26 pad 2: /Source2 -> /PWM1
- R27 pad 1: /Gate4 -> +12V
- R27 pad 2: /Source4 -> /PWM1
- R3 pad 1: Net-(Q2-Pad2) -> /Gate3
- R3 pad 2: /RL2 -> /Source3
- R4 pad 1: +12V -> /Gate4
- R4 pad 2: /PWM3 -> /Source3
- R5 pad 1: Net-(Q5-Pad2) -> /Gate5
- R5 pad 2: /RL3 -> /Source5
- R6 pad 1: +12V -> /Gate6
- R6 pad 2: /PWM2 -> /Source6
- R7 pad 1: +12V -> /Gate7
- R7 pad 2: /PWM1 -> /Source7
- R8 pad 1: Net-(R10-Pad2) -> /Gate8
- R8 pad 2: /Source2 -> /Source7
- R9 pad 1: Net-(R12-Pad2) -> Net-(JP5-Pad3)
- R9 pad 2: LINE -> /Vinv-
- TP1 pad 1: /Source4 -> /Source1
- TP2 pad 1: /Gate4 -> /Gate1
- TP3 pad 1: /Source3 -> /Source2
- TP4 pad 1: /Gate3 -> /Gate2
- TP5 pad 1: /Source2 -> /Source3
- TP6 pad 1: /Gate2 -> /Gate3
- TP7 pad 1: /Source1 -> /Source3
- TP8 pad 1: /Gate1 -> /Gate4
- U2 pad 1: Net-(R16-Pad1) -> Net-(R17-Pad1)
- U2 pad 4: /Vm_in -> /Vm_tapOut
Routing:
- net Net-(C12-Pad2): track 307.5 -> 0.00 mm, vias 2 -> 0
- net Net-(J4-Pad1): track 0.00 -> 306.7 mm
- net /Source7: track 0.00 -> 284.8 mm, vias 0 -> 2
- net /Source6: track 0.00 -> 265.1 mm
- net /Source4: track 262.9 -> 0.00 mm, vias 1 -> 0
- net Net-(C12-Pad1): track 259.6 -> 0.00 mm, vias 2 -> 0
- net +12L: track 256.0 -> 0.00 mm, vias 6 -> 0
- net /Vboost+: track 0.00 -> 237.6 mm
- net +5V: track 0.00 -> 236.4 mm, vias 0 -> 1
- net GNDREF: track 587.0 -> 377.6 mm, vias 10 -> 16
- net +12V: track 302.0 -> 494.7 mm, vias 6 -> 11
- net /Source2: track 316.7 -> 156.9 mm
- net LINE: track 135.5 -> 0.00 mm
- net Net-(D2-Pad2): track 125.5 -> 0.00 mm
- net Net-(D4-Pad2): track 98.1 -> 0.00 mm
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- removed copper zone on F.Cu, net +12L
- removed copper zone on B.Cu, net +12V
- removed copper zone on F.Cu, net +12V
- removed copper zone on B.Cu, net -12V
- removed copper zone on F.Cu, net -12V
- removed copper zone on B.Cu, net /Source2
- removed copper zone on B.Cu, net /Vinv-
- removed copper zone on B.Cu, net /VtapIn
- removed copper zone on B.Cu, net /VtapOut
- removed copper zone on B.Cu, net LINE
- removed copper zone on B.Cu, net NEUT
- removed copper zone on F.Cu, net NEUT
- removed copper zone on F.Cu, net Net-(D2-Pad2)
- removed copper zone on F.Cu, net Net-(D3-Pad2)
- removed copper zone on F.Cu, net Net-(D4-Pad2)
Other:
- board size 259.7 x 125.1 mm -> 308.6 x 115.6 mm
- net class Default: clearance 0.762 -> 0.2; trace_width 0.762 -> 0.25; via_dia 1.524 -> 0.8; via_drill 0.8 -> 0.4
- net class High Voltage removed
- rule pad_to_mask_clearance: 0.2 -> 0
- rule trace_clearance: 0.762 -> 0.2
- board text added: "+12"
- board text added: "+5"
- board text added: "-12"
- board text added: "BI"
- board text added: "BO"
- board text added: "Boost"
- board text added: "OUT"
- board text added: "Out"
- board text added: "S5"
- board text added: "S6"
- board text added: "S7"
- board text added: "S8"
- board text removed: "1"
- board text removed: "2"
- board text removed: "3"
- board text removed: "4"
- board text removed: "G"
- board text removed: "I"
- board text removed: "INV"
- board text removed: "O"
- board text removed: "S"
