File: estabilizador.kicad_pcb (KiCad board)
At the start: 2 copper layers, 259.7 x 125.1 mm, 91 parts, among them J1 Tensão de Entrada, J10 Driver, J11 Tensão do Estágio de Reles, J12 Tensão do Estágio do Inversor, J13 Tensão de Saída Total, J14 Tensão de Medição, J15 Tap AUX2, J2 Autotransformador, J3 Comandos Reles, J4 Tap AUX1, J5 Comandos PWMs, J6 Fonte Aux, J7 Driver, J8 Driver, J9 Driver, K1 RT42xxxx, K2 RT42xxxx, K3 RT42xxxx, Q1 BC517, Q2 BC517, Q3 IRF840N, Q4 IRF840N, Q5 BC517, Q6 IRF840N, Q7 IRF840N, U1 LV20-P, U2 LV25-P

Commit message: Modificação da PCB
Parts:
- removed C14, C15: 1uF, Capacitor_THT:C_Rect_L29.0mm_W7.6mm_P27.50mm_MKT
- removed C2, C3: 1000uF, Capacitor_THT:CP_Radial_D18.0mm_P7.50mm
- removed C4: 390nF, Capacitor_THT:C_Rect_L26.5mm_W7.0mm_P22.50mm_MKS4
- removed C5: 690nF, Capacitor_THT:C_Rect_L29.0mm_W7.6mm_P27.50mm_MKT
- removed D2, D3, D4: 1N4148, Diode_THT:D_DO-35_SOD27_P7.62mm_Horizontal
- removed JP8, JP9: Jumper_NO_Small, Connector_PinHeader_2.54mm:PinHeader_1x02_P2.54mm_Vertical
- removed K1: RT42xxxx, Relay:Relay_DPDT_model_A
- removed K2, K3: RT42xxxx, Relay:Relay_DPDT_model_B
- removed R18, R4: 340R, Resistor_SMD:R_1206_3216Metric_Pad1.42x1.75mm_HandSolder
- added J16: Driver, Connector_PinHeader_2.54mm:PinHeader_1x07_P2.54mm_Vertical, F.Cu at (87.0, 145.4)
- added J17: Driver, Connector_PinHeader_2.54mm:PinHeader_1x07_P2.54mm_Vertical, F.Cu at (64.1, 145.4)
- added J18: Driver, Connector_PinHeader_2.54mm:PinHeader_1x07_P2.54mm_Vertical, F.Cu at (41.3, 145.4)
- added J19: Driver, Connector_PinHeader_2.54mm:PinHeader_1x07_P2.54mm_Vertical, F.Cu at (18.4, 145.4)
- added J20: Fonte Aux, Connector_PinHeader_2.54mm:PinHeader_1x03_P2.54mm_Vertical, F.Cu at (26.7, 163.2)
- added J21: Conn_01x03_Female, Connector_PinHeader_2.54mm:PinHeader_1x03_P2.54mm_Vertical, F.Cu at (456.3, 97.6)
- added J22: Tensão de Medição, Connector_PinHeader_2.54mm:PinHeader_1x04_P2.54mm_Vertical, F.Cu at (189.9, 135.3)
- added J23: Medição da Corrente, Connector_PinHeader_2.54mm:PinHeader_1x02_P2.54mm_Vertical, F.Cu at (204.5, 158.8)
- added L2: L_Core_Ferrite, boost_pfc:NEE_45-45, F.Cu at (316.3, 67.4)
- added Q8: IRF840N, boost_pfc:TO-220-3 Heatsink, F.Cu at (380.1, 137.5)
- added R28: 340R, Resistor_SMD:R_1206_3216Metric_Pad1.42x1.75mm_HandSolder, B.Cu at (98.4, 152.4)
- added R29: 340R, Resistor_SMD:R_1206_3216Metric_Pad1.42x1.75mm_HandSolder, B.Cu at (75.6, 152.4)
- added R30: 340R, Resistor_SMD:R_1206_3216Metric_Pad1.42x1.75mm_HandSolder, B.Cu at (75.6, 149.2)
- added R31: 340R, Resistor_SMD:R_1206_3216Metric_Pad1.42x1.75mm_HandSolder, B.Cu at (52.7, 149.2)
- added R32: 340R, Resistor_SMD:R_1206_3216Metric_Pad1.42x1.75mm_HandSolder, B.Cu at (52.7, 152.4)
- added R33: 340R, Resistor_SMD:R_1206_3216Metric_Pad1.42x1.75mm_HandSolder, B.Cu at (29.8, 152.4)
- added R34: 340R, Resistor_SMD:R_1206_3216Metric_Pad1.42x1.75mm_HandSolder, B.Cu at (29.8, 149.2)
- added TP10: TestPoint, Connector_PinHeader_2.54mm:PinHeader_1x01_P2.54mm_Vertical, F.Cu at (17.1, 151.1)
- added TP11: TestPoint, Connector_PinHeader_2.54mm:PinHeader_1x01_P2.54mm_Vertical, F.Cu at (43.8, 151.1)
- added TP12: TestPoint, Connector_PinHeader_2.54mm:PinHeader_1x01_P2.54mm_Vertical, F.Cu at (40.0, 151.1)
- added TP13: TestPoint, Connector_PinHeader_2.54mm:PinHeader_1x01_P2.54mm_Vertical, F.Cu at (66.7, 151.1)
- added TP14: TestPoint, Connector_PinHeader_2.54mm:PinHeader_1x01_P2.54mm_Vertical, F.Cu at (62.9, 151.1)
- added TP15: TestPoint, Connector_PinHeader_2.54mm:PinHeader_1x01_P2.54mm_Vertical, F.Cu at (89.5, 151.1)
- added TP16: TestPoint, Connector_PinHeader_2.54mm:PinHeader_1x01_P2.54mm_Vertical, F.Cu at (85.7, 151.1)
- added TP9: TestPoint, Connector_PinHeader_2.54mm:PinHeader_1x01_P2.54mm_Vertical, F.Cu at (21.0, 151.1)
- C1: value 1000uF -> 2700uF
- C10, C11: moved to F.Cu
- C12: value 2uF -> 100nF; footprint Capacitor_THT:C_Rect_L29.0mm_W7.6mm_P27.50mm_MKT -> Capacitor_SMD:C_0805_2012Metric_Pad1.15x1.40mm_HandSolder
- C13: value 2uF -> 100uF; footprint Capacitor_THT:C_Rect_L29.0mm_W7.6mm_P27.50mm_MKT -> Capacitor_SMD:CP_Elec_8x10
- C6: value 690nF -> 390nF; footprint Capacitor_THT:C_Rect_L29.0mm_W7.6mm_P27.50mm_MKT -> Capacitor_THT:C_Rect_L26.5mm_W7.0mm_P22.50mm_MKS4
- C8: value 100nF -> 690nF; footprint Capacitor_SMD:C_0805_2012Metric_Pad1.15x1.40mm_HandSolder -> Capacitor_THT:C_Rect_L29.0mm_W7.6mm_P27.50mm_MKT; moved to F.Cu
- C9: value 100uF -> 690nF; footprint Capacitor_SMD:CP_Elec_8x10 -> Capacitor_THT:C_Rect_L29.0mm_W7.6mm_P27.50mm_MKT; moved to F.Cu
- D1: value GBU8J -> 3,3 V; footprint Diode_THT:Diode_Bridge_Vishay_KBU -> Diode_SMD:D_SOT-23_ANK
- J10: value Driver -> Comandos PWMs; footprint Connector_PinHeader_2.54mm:PinHeader_1x07_P2.54mm_Vertical -> Connector_PinHeader_2.54mm:PinHeader_1x08_P2.54mm_Vertical
- J11: value Tensão do Estágio de Reles -> Driver; footprint Connector_Phoenix_MSTB:PhoenixContact_MSTBVA_2,5_2-G-5,08_1x02_P5.08mm_Vertical -> Connector_PinHeader_2.54mm:PinHeader_1x07_P2.54mm_Vertical
- J12: value Tensão do Estágio do Inversor -> Driver; footprint Connector_Phoenix_MSTB:PhoenixContact_MSTBVA_2,5_2-G-5,08_1x02_P5.08mm_Vertical -> Connector_PinHeader_2.54mm:PinHeader_1x07_P2.54mm_Vertical
- J13: value Tensão de Saída Total -> Driver; footprint Connector_Phoenix_MSTB:PhoenixContact_MSTBVA_2,5_2-G-5,08_1x02_P5.08mm_Vertical -> Connector_PinHeader_2.54mm:PinHeader_1x07_P2.54mm_Vertical
- J14: value Tensão de Medição -> Driver; footprint Connector_PinHeader_2.54mm:PinHeader_1x04_P2.54mm_Vertical -> Connector_PinHeader_2.54mm:PinHeader_1x07_P2.54mm_Vertical
- J15: value Tap AUX2 -> Comandos PWMs; footprint Connector_Phoenix_MSTB:PhoenixContact_MSTBVA_2,5_4-G-5,08_1x04_P5.08mm_Vertical -> Connector_PinHeader_2.54mm:PinHeader_1x08_P2.54mm_Vertical
- J2: value Autotransformador -> Alimentação ACS712; footprint Connector_Phoenix_MSTB:PhoenixContact_MSTBVA_2,5_5-G-5,08_1x05_P5.08mm_Vertical -> Connector_PinHeader_2.54mm:PinHeader_1x02_P2.54mm_Vertical
- J3: value Comandos Reles -> Tap AUX1; footprint Connector_PinHeader_2.54mm:PinHeader_1x06_P2.54mm_Vertical -> Connector_Phoenix_MSTB:PhoenixContact_MSTBVA_2,5_2-G-5,08_1x02_P5.08mm_Vertical
- J4: value Tap AUX1 -> Screw_Terminal_01x02
- J5: value Comandos PWMs -> Sensor de Corrente; footprint Connector_PinHeader_2.54mm:PinHeader_1x08_P2.54mm_Vertical -> Connector_Phoenix_MSTB:PhoenixContact_MSTBVA_2,5_2-G-5,08_1x02_P5.08mm_Vertical
- J6: value Fonte Aux -> Tensão do Estabilizador; footprint Connector_PinHeader_2.54mm:PinHeader_1x03_P2.54mm_Vertical -> Connector_Phoenix_MSTB:PhoenixContact_MSTBVA_2,5_2-G-5,08_1x02_P5.08mm_Vertical
- J7: value Driver -> Tensão do Estágio do Inversor; footprint Connector_PinHeader_2.54mm:PinHeader_1x07_P2.54mm_Vertical -> Connector_Phoenix_MSTB:PhoenixContact_MSTBVA_2,5_2-G-5,08_1x02_P5.08mm_Vertical
- J8: value Driver -> Tensão de Saída Total; footprint Connector_PinHeader_2.54mm:PinHeader_1x07_P2.54mm_Vertical -> Connector_Phoenix_MSTB:PhoenixContact_MSTBVA_2,5_2-G-5,08_1x02_P5.08mm_Vertical
- J9: value Driver -> Tensão de Saída do Boost; footprint Connector_PinHeader_2.54mm:PinHeader_1x07_P2.54mm_Vertical -> Connector_Phoenix_MSTB:PhoenixContact_MSTBVA_2,5_2-G-5,08_1x02_P5.08mm_Vertical
- JP3: value Jumper_NO_Small -> Jumper_3_Bridged12; footprint Connector_PinHeader_2.54mm:PinHeader_1x02_P2.54mm_Vertical -> Connector_PinHeader_2.54mm:PinHeader_1x03_P2.54mm_Vertical
- JP4: value Jumper_3_Bridged12 -> Jumper_NO_Small; footprint Connector_PinHeader_2.54mm:PinHeader_1x03_P2.54mm_Vertical -> Connector_PinHeader_2.54mm:PinHeader_1x02_P2.54mm_Vertical
- L1: footprint Inductors:Inductor_EE4220 -> boost_pfc:NEE_30-14
- Q1, Q2: value BC517 -> IRG4PF50W; footprint Package_TO_SOT_THT:TO-92_Inline_Wide -> Package_TO_SOT_THT:TO-247-3_Vertical
- Q3, Q4: value IRF840N -> IRG4PF50W; footprint transistors:TO-220-3 Heatsink -> Package_TO_SOT_THT:TO-247-3_Vertical
- Q5: value BC517 -> IRF840N; footprint Package_TO_SOT_THT:TO-92_Inline_Wide -> boost_pfc:TO-220-3 Heatsink
- Q6, Q7: footprint transistors:TO-220-3 Heatsink -> boost_pfc:TO-220-3 Heatsink
- R1, R3, R5: value 100K -> 10k; moved to F.Cu
- R10: value 10K -> 3K3; footprint Resistor_THT:R_Axial_DIN0414_L11.9mm_D4.5mm_P15.24mm_Horizontal -> Resistor_THT:R_Axial_DIN0309_L9.0mm_D3.2mm_P12.70mm_Horizontal
- R11: value 3K3 -> 10K; footprint Resistor_THT:R_Axial_DIN0309_L9.0mm_D3.2mm_P12.70mm_Horizontal -> Resistor_THT:R_Axial_DIN0414_L11.9mm_D4.5mm_P15.24mm_Horizontal
- R14: value 10k -> 2K2
- R15, R16: value 10k -> 10K; footprint Resistor_THT:R_Axial_DIN0414_L11.9mm_D4.5mm_P15.24mm_Horizontal -> Resistor_THT:R_Axial_DIN0207_L6.3mm_D2.5mm_P10.16mm_Horizontal
- R17: value 340R -> 567; footprint Resistor_SMD:R_1206_3216Metric_Pad1.42x1.75mm_HandSolder -> Resistor_SMD:R_0805_2012Metric_Pad1.15x1.40mm_HandSolder; moved to F.Cu
- R2, R6, R7: value 340R -> 10k; footprint Resistor_SMD:R_1206_3216Metric_Pad1.42x1.75mm_HandSolder -> Resistor_SMD:R_0805_2012Metric_Pad1.15x1.40mm_HandSolder; moved to F.Cu
- R21, R22, R23: value 10K -> 340R; footprint Resistor_SMD:R_0805_2012Metric_Pad1.15x1.40mm_HandSolder -> Resistor_SMD:R_1206_3216Metric_Pad1.42x1.75mm_HandSolder
- R24, R25, R26, R27: value 10k -> 340R; footprint Resistor_SMD:R_0805_2012Metric_Pad1.15x1.40mm_HandSolder -> Resistor_SMD:R_1206_3216Metric_Pad1.42x1.75mm_HandSolder
- R8, R9: value 10K -> 10k; footprint Resistor_THT:R_Axial_DIN0414_L11.9mm_D4.5mm_P15.24mm_Horizontal -> Resistor_SMD:R_0805_2012Metric_Pad1.15x1.40mm_HandSolder
- moved Q3 401.9 mm to (434.9, 87.3)
- moved J5 352.8 mm to (424.2, 113.0), turned to 0 degrees
- moved R7 340.6 mm to (385.4, 147.0)
- moved R6 331.6 mm to (398.7, 155.3)
- moved Q7 328.8 mm to (429.4, 78.2)
- moved Q4 326.1 mm to (405.5, 114.6)
- moved R2 309.5 mm to (423.1, 140.1)
- moved R8 303.1 mm to (436.2, 129.0), turned to 0 degrees
- moved R15 302.2 mm to (457.7, 77.4), turned to 0 degrees
- moved Q6 297.1 mm to (352.0, 141.4)
- moved R10 289.3 mm to (433.2, 93.1), turned to 0 degrees
- moved JP3 281.4 mm to (436.2, 120.1), turned to 0 degrees
- moved JP6 277.3 mm to (405.2, 148.0), turned to 0 degrees
- moved R17 276.8 mm to (390.0, 118.6)
- moved JP5 267.3 mm to (418.7, 131.2), turned to 0 degrees
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Connections:
- C1 pad 1: /HI_in_inv -> /Vboost+
- C1 pad 2: /LO_in_inv -> /Source3
- C12 pad 1: Net-(C12-Pad1) -> -12V
- C12 pad 2: Net-(C12-Pad2) -> +12V
- C13 pad 1: /Source3 -> +12V
- C13 pad 2: /Source4 -> -12V
- C6 pad 1: Net-(C5-Pad1) -> Net-(C6-Pad1)
- C6 pad 2: /Source2 -> Net-(C6-Pad2)
- C7 pad 1: Net-(C4-Pad2) -> Net-(C6-Pad2)
- C7 pad 2: /Source2 -> /Source6
- C8 pad 1: -12V -> Net-(C8-Pad1)
- C8 pad 2: +12V -> /Source6
- C9 pad 1: +12V -> Net-(C8-Pad1)
- C9 pad 2: -12V -> /Source6
- D1 pad 1: /HI_in_inv -> /Vm_acs712
- D1 pad 2: /VauxA -> GNDREF
- J1 pad 2: LINE -> /VtapOut
- J10 pad 1: /Gate1 -> /PWM1
- J10 pad 2: /Source1 -> GNDREF
- J10 pad 3: Net-(J10-Pad3) -> /PWM2
- J10 pad 5: +12V -> /PWM3
- J10 pad 6: /PWM1 -> GNDREF
- J10 pad 7: GNDREF -> /PWM4
- J11 pad 1: NEUT -> /Gate4
- J11 pad 2: /VtapOut -> /Source3
- J12 pad 1: /Vinv- -> /Gate3
- J12 pad 2: /Source2 -> /Source3
- J13 pad 1: /Source2 -> /Gate2
- J13 pad 2: NEUT -> /Source2
- J14 pad 1: GNDREF -> /Gate1
- J14 pad 2: /Vm_out -> /Source1
- J14 pad 3: GNDREF -> Net-(J14-Pad3)
- J14 pad 4: /Vm_in -> GNDREF
- J15 pad 1: Net-(C12-Pad1) -> /PWM5
- J15 pad 2: Net-(C12-Pad2) -> GNDREF
- J15 pad 3: /Source3 -> /PWM6
- J15 pad 4: /Source4 -> GNDREF
- J2 pad 1: /Vtap1 -> +5V
- J2 pad 2: /VtapIn -> GNDREF
- J3 pad 1: /RL1 -> /VauxA
- J3 pad 2: GNDREF -> /Source2
- J4 pad 1: /VauxA -> Net-(J4-Pad1)
- J4 pad 2: /VauxB -> /Source7
- J5 pad 1: /PWM1 -> Net-(J5-Pad1)
- J5 pad 2: GNDREF -> /Source1
- J6 pad 1: +12V -> NEUT
- J6 pad 2: GNDREF -> /VtapOut
- J7 pad 1: /Gate4 -> /Vinv-
- J7 pad 2: /Source4 -> /Source6
- J8 pad 1: /Gate3 -> /Source6
- J8 pad 2: /Source3 -> NEUT
- J9 pad 1: /Gate2 -> /Vboost+
- J9 pad 2: /Source2 -> /Source3
- JP1 pad 1: Net-(C12-Pad2) -> Net-(J4-Pad1)
- JP1 pad 2: /HI_in_inv -> /Vboost+
- JP2 pad 1: /Source3 -> /Source7
- JP2 pad 2: /LO_in_inv -> /Source3
- JP3 pad 1: /VtapOut -> Net-(C8-Pad1)
- JP4 pad 1: Net-(C5-Pad1) -> /VtapOut
- JP6 pad 3: /Source2 -> /Source6
- L1 pad 1: /Source1 -> Net-(J5-Pad1)
- L1 pad 2: /Vinv- -> /VauxA
- Q1 pad 1: Net-(D2-Pad2) -> /Gate1
- Q1 pad 2: Net-(Q1-Pad2) -> /Vboost+
- Q1 pad 3: GNDREF -> /Source1
- Q2 pad 1: Net-(D3-Pad2) -> /Gate2
- Q2 pad 2: Net-(Q2-Pad2) -> /Vboost+
- Q2 pad 3: GNDREF -> /Source2
- Q3 pad 1: /Gate1 -> /Gate3
- Q3 pad 2: Net-(C12-Pad2) -> /Source1
- Q3 pad 3: /Source1 -> /Source3
- Q4 pad 1: /Gate3 -> /Gate4
- Q4 pad 2: /Source1 -> /Source2
- Q5 pad 1: Net-(D4-Pad2) -> /Gate5
- Q5 pad 2: Net-(Q5-Pad2) -> Net-(J4-Pad1)
- Q5 pad 3: GNDREF -> /Source5
- Q6 pad 1: /Gate2 -> /Gate6
- Q6 pad 2: Net-(C12-Pad1) -> Net-(J4-Pad1)
- Q6 pad 3: /Source2 -> /Source6
- Q7 pad 1: /Gate4 -> /Gate7
- Q7 pad 2: /Source2 -> /Source5
- Q7 pad 3: /Source4 -> /Source7
- R1 pad 1: Net-(Q1-Pad2) -> /Gate1
- R1 pad 2: /RL1 -> /Source1
- R10 pad 1: Net-(R10-Pad1) -> Net-(JP5-Pad3)
- R10 pad 2: Net-(R10-Pad2) -> /Vinv-
- R11 pad 1: Net-(JP5-Pad3) -> Net-(R11-Pad1)
- R11 pad 2: /Vinv- -> /Source6
- R12 pad 2: Net-(R12-Pad2) -> Net-(R11-Pad1)
- R13 pad 2: Net-(R10-Pad1) -> Net-(R12-Pad1)
- R14 pad 1: Net-(R14-Pad1) -> Net-(JP5-Pad1)
- R14 pad 2: Net-(R12-Pad1) -> Net-(R13-Pad1)
- R15 pad 1: Net-(JP5-Pad1) -> Net-(R15-Pad1)
- R15 pad 2: Net-(R13-Pad1) -> /Vboost+
- R16 pad 2: Net-(R14-Pad1) -> Net-(R15-Pad1)
- R17 pad 1: +12V -> /Vm_acs712
- R17 pad 2: /PWM4 -> Net-(J21-Pad2)
- R19 pad 2: /PWM2 -> /PWM4
- R2 pad 1: +12V -> /Gate2
- R2 pad 2: /PWM4 -> /Source2
- R20 pad 2: /PWM1 -> /PWM4
- R21 pad 1: /RL1 -> +12V
- R21 pad 2: +12L -> /PWM3
- R22 pad 1: /RL2 -> +12V
- R22 pad 2: +12L -> /PWM3
- R23 pad 1: /RL3 -> +12V
- R23 pad 2: +12L -> /PWM2
- R24 pad 1: /Gate1 -> +12V
- R24 pad 2: /Source1 -> /PWM2
- R25 pad 1: /Gate3 -> +12V
- R25 pad 2: /Source3 -> /PWM1
- R26 pad 1: /Gate2 -> +12V
- R26 pad 2: /Source2 -> /PWM1
- R27 pad 1: /Gate4 -> +12V
- R27 pad 2: /Source4 -> /PWM8
- R3 pad 1: Net-(Q2-Pad2) -> /Gate3
- R3 pad 2: /RL2 -> /Source3
- R5 pad 1: Net-(Q5-Pad2) -> /Gate4
- R5 pad 2: /RL3 -> /Source3
- R6 pad 1: +12V -> /Gate5
- R6 pad 2: /PWM2 -> /Source5
- R7 pad 1: +12V -> /Gate7
- R7 pad 2: /PWM1 -> /Source7
- R8 pad 1: Net-(R10-Pad2) -> /Gate6
- R8 pad 2: /Source2 -> /Source6
- R9 pad 1: Net-(R12-Pad2) -> /Gate8
- R9 pad 2: LINE -> /Source7
- TP1 pad 1: /Source4 -> /Source1
- TP2 pad 1: /Gate4 -> /Gate1
- TP3 pad 1: /Source3 -> /Source2
- TP4 pad 1: /Gate3 -> /Gate2
- TP5 pad 1: /Source2 -> /Source3
- TP6 pad 1: /Gate2 -> /Gate3
- TP7 pad 1: /Source1 -> /Source3
- TP8 pad 1: /Gate1 -> /Gate4
- U2 pad 3: NEUT -> /Source3
- U2 pad 4: /Vm_in -> /Vm_boost
Routing:
- net GNDREF: track 587.0 -> 111.1 mm, vias 10 -> 0
- net NEUT: track 411.5 -> 0.00 mm
- net /Source2: track 316.7 -> 5.72 mm
- net Net-(C12-Pad2): track 307.5 -> 0.00 mm, vias 2 -> 0
- net /Source4: track 262.9 -> 0.00 mm, vias 1 -> 0
- net /Source3: track 271.2 -> 11.4 mm
- net Net-(C12-Pad1): track 259.6 -> 0.00 mm, vias 2 -> 0
- net +12L: track 256.0 -> 0.00 mm, vias 6 -> 0
- net -12V: track 248.8 -> 73.2 mm, vias 2 -> 0
- net /Vinv-: track 174.4 -> 0.00 mm
- net LINE: track 135.5 -> 0.00 mm
- net +12V: track 302.0 -> 176.1 mm, vias 6 -> 4
- net Net-(D2-Pad2): track 125.5 -> 0.00 mm
- net /Source1: track 122.3 -> 5.72 mm
- net /VtapOut: track 105.9 -> 0.00 mm
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- removed copper zone on F.Cu, net +12L
- removed copper zone on B.Cu, net +12V
- removed copper zone on F.Cu, net +12V
- removed copper zone on B.Cu, net -12V
- removed copper zone on F.Cu, net -12V
- removed copper zone on B.Cu, net /Source2
- removed copper zone on B.Cu, net /Vinv-
- removed copper zone on B.Cu, net /VtapIn
- removed copper zone on B.Cu, net /VtapOut
- removed copper zone on B.Cu, net GNDREF
- removed copper zone on F.Cu, net GNDREF
- removed copper zone on B.Cu, net LINE
- removed copper zone on B.Cu, net NEUT
- removed copper zone on F.Cu, net NEUT
- removed copper zone on F.Cu, net Net-(D2-Pad2)
- removed copper zone on F.Cu, net Net-(D3-Pad2)
- removed copper zone on F.Cu, net Net-(D4-Pad2)
Other:
- board outline removed
- net class Default: clearance 0.762 -> 0.2; trace_width 0.762 -> 0.25; via_dia 1.524 -> 0.8; via_drill 0.8 -> 0.4
- net class High Voltage removed
- rule pad_to_mask_clearance: 0.2 -> 0
- rule trace_clearance: 0.762 -> 0.2
- board text removed: "+"
- board text removed: "-"
- board text removed: "1"
- board text removed: "2"
- board text removed: "3"
- board text removed: "4"
- board text removed: "Conversor CA-CA Híbrido"
- board text removed: "Câmpus Florianópolis"
- board text removed: "G"
- board text removed: "I"
- board text removed: "IN"
- board text removed: "INV"
- board text removed: "Instituto Federal"
- board text removed: "L"
- board text removed: "N"
- board text removed: "O"
- board text removed: "S"
- board text removed: "S1"
- board text removed: "S2"
- board text removed: "S3"
- board text removed: "S4"
- board text removed: "Santa Catarina"
- board text removed: "TapOut"
- board text removed: "ΔV"

Commit message: Modificação da PCB
Parts:
- added C14: 100nF, Capacitor_SMD:C_0805_2012Metric_Pad1.15x1.40mm_HandSolder, F.Cu at (374.0, 250.8)
- added C15: 100uF, Capacitor_SMD:CP_Elec_8x10, F.Cu at (389.4, 247.4)
- added D1: 3,3 V, Diode_SMD:D_SOT-23_ANK, F.Cu at (373.9, 257.5)
- added J2: Alimentação LTSP 25-NP, Connector_PinHeader_2.54mm:PinHeader_1x02_P2.54mm_Vertical, F.Cu at (369.3, 251.7)
- added J20: Tensão de Medição, Connector_PinHeader_2.54mm:PinHeader_1x08_P2.54mm_Vertical, F.Cu at (327.7, 163.8)
- added R15: 10K, Resistor_THT:R_Axial_DIN0414_L11.9mm_D4.5mm_P15.24mm_Horizontal, F.Cu at (297.8, 75.6)
- added R16: 10K, Resistor_THT:R_Axial_DIN0414_L11.9mm_D4.5mm_P15.24mm_Horizontal, F.Cu at (295.3, 95.2)
- added R19: 10K, Resistor_THT:R_Axial_DIN0207_L6.3mm_D2.5mm_P10.16mm_Horizontal, F.Cu at (311.8, 93.3)
- added R20: 10K, Resistor_THT:R_Axial_DIN0207_L6.3mm_D2.5mm_P10.16mm_Horizontal, F.Cu at (315.0, 93.3)
- added R37: 56, Resistor_THT:R_Axial_DIN0207_L6.3mm_D2.5mm_P10.16mm_Horizontal, F.Cu at (-14.6, 107.3)
- added R38: 567, Resistor_THT:R_Axial_DIN0207_L6.3mm_D2.5mm_P10.16mm_Horizontal, F.Cu at (-24.1, 118.7)
- added U3: LTSP_25-NP, Sensor_Current:LEM_LTSR-NP, F.Cu at (34.9, 135.9)
- added U4: LV25-P, Sensor_Voltage:LEM_LV25-P, F.Cu at (315.0, 107.3)
- R17: renamed from R15; footprint Resistor_THT:R_Axial_DIN0207_L6.3mm_D2.5mm_P10.16mm_Horizontal -> Resistor_THT:R_Axial_DIN0414_L11.9mm_D4.5mm_P15.24mm_Horizontal
- R18: renamed from R16; footprint Resistor_THT:R_Axial_DIN0207_L6.3mm_D2.5mm_P10.16mm_Horizontal -> Resistor_THT:R_Axial_DIN0414_L11.9mm_D4.5mm_P15.24mm_Horizontal
- moved Q1 377.9 mm to (48.3, 124.5)
- moved Q3 342.9 mm to (94.0, 124.5)
- moved Q2 334.4 mm to (71.1, 124.5)
- moved C1 321.2 mm to (87.6, 94.0)
- moved Q4 288.8 mm to (116.8, 124.5)
- moved L1 280.0 mm to (36.8, 94.6), turned to 90 degrees
- moved J3 261.7 mm to (22.9, 69.2), turned to 90 degrees
- moved Q5 250.0 mm to (139.7, 126.4)
- moved Q7 248.7 mm to (185.4, 126.4)
- moved JP3 227.0 mm to (216.5, 62.9), turned to 90 degrees
- moved J8 195.1 mm to (311.8, 62.2)
- moved Q6 190.1 mm to (162.6, 126.4)
- moved C13 187.4 mm to (286.4, 182.9)
- moved Q8 172.2 mm to (208.3, 126.4)
- moved L2 171.5 mm to (148.0, 100.3), turned to 90 degrees
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- renumbered J15 to J10, J16 to J15, J17 to J16, J18 to J17, J19 to J18, J20 to J19, J6 to J5, J7 to J6, J8 to J7, J9 to J8, J10 to J9, R19 to R21, R20 to R22, R21 to R23, R22 to R24, R23 to R25, R24 to R26, R25 to R27, R26 to R28, R27 to R29, R28 to R30, R29 to R31, R30 to R32, R31 to R33, R32 to R34, R33 to R35, R34 to R36
Connections:
- L1 pad 1: Net-(J5-Pad1) -> Net-(L1-Pad1)
- R17 pad 2: /Vboost+ -> Net-(R16-Pad1)
- U2 pad 3: /Source3 -> NEUT
- U2 pad 4: /Vm_boost -> /Vm_tapOut
Routing:
- net /Source6: track 5.72 -> 278.4 mm
- net NEUT: track 0.00 -> 233.5 mm
- net GNDREF: track 111.1 -> 313.2 mm, vias 0 -> 16
- net /Vinv-: track 0.00 -> 160.1 mm
- net /Source3: track 11.4 -> 102.2 mm
- net /Source5: track 5.72 -> 90.0 mm
- net /Gate1: track 6.24 -> 40.4 mm
- net Net-(J4-Pad1): track 0.00 -> 27.7 mm
- net /Source7: track 11.4 -> 37.7 mm
- net Net-(C6-Pad2): track 0.00 -> 26.2 mm
- net Net-(C8-Pad1): track 0.00 -> 22.3 mm
- net /Vboost+: track 0.00 -> 21.0 mm
- net Net-(C6-Pad1): track 0.00 -> 19.7 mm
- net /Source2: track 5.72 -> 25.0 mm
- net /Source1: track 5.72 -> 25.0 mm
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
Commit message: Modificação do esquemático e PCB
Parts:
- removed the D1 at (470.1, 100.8)
- removed the J2 at (369.3, 251.7)
- removed J21: Conn_01x03_Female, Connector_PinHeader_2.54mm:PinHeader_1x03_P2.54mm_Vertical
- removed J22: Tensão de Medição, Connector_PinHeader_2.54mm:PinHeader_1x04_P2.54mm_Vertical
- removed J23: Medição da Corrente, Connector_PinHeader_2.54mm:PinHeader_1x02_P2.54mm_Vertical
- removed the J5 at (424.2, 113.0)
- removed JP7: Jumper_NO_Small, Connector_PinHeader_2.54mm:PinHeader_1x02_P2.54mm_Vertical
- removed the R17 at (390.0, 118.6)
- C10, C11, C12, C13, C14, C15, R1, R2, R3, R5, R6, R7, R8, R9: moved to B.Cu
- D1: footprint Diode_SMD:D_SOT-23_ANK -> Diode_THT:D_DO-35_SOD27_P7.62mm_Horizontal
- R38: value 567 -> 75
- moved R8 367.0 mm to (69.2, 130.8)
- moved R6 353.2 mm to (46.4, 130.8)
- moved J3 301.8 mm to (324.5, 79.4), turned to 270 degrees
- moved R7 293.8 mm to (92.1, 130.8)
- moved R37 285.9 mm to (271.3, 103.4), turned to 180 degrees
- moved R9 274.0 mm to (114.9, 130.8)
- moved R38 263.9 mm to (239.4, 104.8), turned to 0 degrees
- moved L1 249.1 mm to (283.8, 62.2), turned to 0 degrees
- moved U3 221.6 mm to (251.8, 90.8), turned to 90 degrees
- moved C15 202.7 mm to (216.5, 141.6)
- moved D1 201.1 mm to (239.4, 108.0)
- moved C14 196.1 mm to (216.5, 134.0), turned to 180 degrees
- moved R1 195.9 mm to (245.1, 130.2)
- moved TP5 195.6 mm to (292.1, 144.1)
- moved TP6 195.6 mm to (288.3, 144.1)
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Connections:
- J20 pad 1: GNDREF -> /Vm_out
- J20 pad 2: /Vm_LTSP_25-NP -> GNDREF
- J20 pad 3: GNDREF -> /Vm_tapOut
- J20 pad 4: /Vm_boost -> GNDREF
- J20 pad 5: GNDREF -> /Vm_boost
- J20 pad 6: /Vm_out -> GNDREF
- J20 pad 7: GNDREF -> /Vm_LTSP_25-NP
- J20 pad 8: /Vm_tapOut -> GNDREF
Routing:
- net +12V: track 176.1 -> 494.7 mm, vias 4 -> 11
- net Net-(J4-Pad1): track 27.7 -> 295.8 mm
- net /Source7: track 37.7 -> 284.8 mm, vias 0 -> 2
- net /Vboost+: track 21.0 -> 226.0 mm
- net NEUT: track 233.5 -> 419.6 mm
- net +5V: track 57.0 -> 236.4 mm, vias 0 -> 1
- net -12V: track 73.2 -> 246.5 mm, vias 0 -> 3
- net /VtapOut: track 13.3 -> 167.8 mm
- net /Source3: track 102.2 -> 256.3 mm
- net /Source1: track 25.0 -> 119.7 mm
- net /Source2: track 25.0 -> 116.8 mm
- net /Vm_LTSP_25-NP: track 0.00 -> 86.2 mm
- net GNDREF: track 313.2 -> 377.6 mm
- net /Vm_out: track 0.00 -> 58.6 mm
- net Net-(L1-Pad1): track 0.00 -> 37.2 mm
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Other:
- board outline added: 308.6 x 115.6 mm
- board text added: "Conversor CA-CA Híbrido"
- board text added: "Câmpus Florianópolis"
- board text added: "Instituto Federal"
- board text added: "Santa Catarina"

Commit message: Alteração das labels/Finalização PCB
Parts:
- J2: value Alimentação ACS712 -> Alimentação LTSP 25-NP
- moved C1 7.62 mm to (261.0, 62.2)
- moved R36 1.40 mm to (271.1, 104.8)
- renumbered R11 to R10, R12 to R11, R13 to R12, R14 to R13, R15 to R14, R16 to R15, R17 to R16, R18 to R17, R19 to R18, R20 to R19, R21 to R20, R22 to R21, R23 to R22, R24 to R23, R25 to R24, R26 to R25, R27 to R26, R28 to R27, R29 to R28, R30 to R29, R31 to R30, R32 to R31, R33 to R32, R34 to R33, R35 to R34, R36 to R35, R37 to R36, R38 to R37, R5 to R4, R6 to R5, R8 to R6, R9 to R8, R10 to R9, U4 to U3, U3 to U4
Routing:
- net /Source2: track 116.8 -> 156.9 mm
- net /Vboost+: track 226.0 -> 237.6 mm
- net Net-(J4-Pad1): track 295.8 -> 306.7 mm
- net /Source6: track 254.5 -> 265.1 mm
- net NEUT: track 419.6 -> 427.6 mm
- net Net-(R36-Pad2): track 4.98 -> 11.3 mm
- net /Vinv-: track 167.8 -> 172.9 mm
- net /Source3: track 256.3 -> 251.9 mm
- net /Vm_out: track 58.6 -> 60.4 mm
- net Net-(R36-Pad1): track 31.2 -> 32.8 mm
- net /Source5: track 86.2 -> 87.7 mm
- added copper zone on B.Cu, net GNDREF
- added copper zone on F.Cu, net GNDREF
Other:
- board text added: "+"
- board text added: "+12"
- board text added: "+5"
- board text added: "-"
- board text added: "-12"
- board text added: "BI"
- board text added: "BO"
- board text added: "Boost"
- board text added: "IN"
- board text added: "L"
- board text added: "N"
- board text added: "OUT"
- board text added: "Out"
- board text added: "S1"
- board text added: "S2"
- board text added: "S3"
- board text added: "S4"
- board text added: "S5"
- board text added: "S6"
- board text added: "S7"
- board text added: "S8"
- board text added: "TapOut"
- board text added: "ΔV"

Commit message: Modificação drivers e chaves
Parts:
- removed the J10 at (84.5, 156.2)
- removed the J16 at (90.8, 138.4)
- removed the J17 at (67.9, 138.4)
- removed the J18 at (45.1, 138.4)
- removed the R15 at (200.7, 95.2)
- removed the R16 at (195.6, 80.0)
- removed the R17 at (190.5, 95.2)
- removed the R18 at (217.2, 93.3)
- removed the R19 at (220.3, 93.3)
- removed the R31 at (102.2, 142.2)
- removed R34, R35: 340R, Resistor_SMD:R_1206_3216Metric_Pad1.42x1.75mm_HandSolder
- removed R37: 75, Resistor_THT:R_Axial_DIN0207_L6.3mm_D2.5mm_P10.16mm_Horizontal
- added C1: 4700uF, Capacitor_THT:CP_Radial_D18.0mm_P7.50mm, F.Cu at (220.1, 87.8)
- added C3: 910nF, Capacitor_THT:C_Rect_L29.0mm_W7.6mm_P27.50mm_MKT, F.Cu at (115.7, 68.7)
- added C8: 100uF, Capacitor_SMD:CP_Elec_8x10, F.Cu at (241.4, 97.4)
- added C9: 100nF, Capacitor_SMD:C_0805_2012Metric_Pad1.15x1.40mm_HandSolder, F.Cu at (249.2, 97.4)
- added J11: Comandos Inversor, Connector_PinHeader_2.54mm:PinHeader_1x08_P2.54mm_Vertical, F.Cu at (93.6, 156.2)
- added J12: Driver, Connector_PinHeader_2.54mm:PinHeader_1x07_P2.54mm_Vertical, F.Cu at (122.8, 138.4)
- added J13: Driver, Connector_PinHeader_2.54mm:PinHeader_1x07_P2.54mm_Vertical, F.Cu at (99.9, 138.4)
- added J14: Driver, Connector_PinHeader_2.54mm:PinHeader_1x07_P2.54mm_Vertical, F.Cu at (77.1, 138.4)
- added R14: 1k5, Resistor_THT:R_Axial_DIN0309_L9.0mm_D3.2mm_P12.70mm_Horizontal, F.Cu at (206.8, 93.3)
- added R23: 340R, Resistor_SMD:R_1206_3216Metric_Pad1.42x1.75mm_HandSolder, B.Cu at (134.2, 142.2)
- added R24: 340R, Resistor_SMD:R_1206_3216Metric_Pad1.42x1.75mm_HandSolder, B.Cu at (134.2, 145.5)
- added R25: 340R, Resistor_SMD:R_1206_3216Metric_Pad1.42x1.75mm_HandSolder, B.Cu at (111.3, 145.7)
- added R26: 340R, Resistor_SMD:R_1206_3216Metric_Pad1.42x1.75mm_HandSolder, B.Cu at (111.3, 142.2)
- added R27: 340R, Resistor_SMD:R_1206_3216Metric_Pad1.42x1.75mm_HandSolder, B.Cu at (88.5, 142.2)
- C2: renamed from C1; value 2700uF -> 4700uF
- C4: renamed from C9; value 690nF -> 910nF
- C5: renamed from C8; value 690nF -> 910nF
- C6, C7: value 390nF -> 750nF
- J2: value Alimentação LTSP 25-NP -> Fonte Aux2
- J5: renamed from J9; value Comandos PWMs -> Comandos Boost
- L2: footprint boost_pfc:NEE_45-45 -> boost_pfc:NEE_42-20
- Q1, Q2, Q3, Q4: value IRG4PF50W -> IRF540N; footprint Package_TO_SOT_THT:TO-247-3_Vertical -> boost_pfc:TO-220-3 Heatsink
- R10, R11: value 10K -> 5k6; footprint Resistor_THT:R_Axial_DIN0414_L11.9mm_D4.5mm_P15.24mm_Horizontal -> Resistor_THT:R_Axial_DIN0411_L9.9mm_D3.6mm_P15.24mm_Horizontal
- R12: value 10k -> 5k6; footprint Resistor_THT:R_Axial_DIN0414_L11.9mm_D4.5mm_P15.24mm_Horizontal -> Resistor_THT:R_Axial_DIN0411_L9.9mm_D3.6mm_P15.24mm_Horizontal
- R13: value 2K2 -> 5k6; footprint Resistor_THT:R_Axial_DIN0414_L11.9mm_D4.5mm_P15.24mm_Horizontal -> Resistor_THT:R_Axial_DIN0411_L9.9mm_D3.6mm_P15.24mm_Horizontal
- R31: renamed from R36; value 56 -> 200; footprint Resistor_THT:R_Axial_DIN0207_L6.3mm_D2.5mm_P10.16mm_Horizontal -> Resistor_SMD:R_1206_3216Metric_Pad1.42x1.75mm_HandSolder; moved to B.Cu
- R32: value 340R -> 10k
- R33: value 340R -> 15k
- R9: value 3K3 -> 750; footprint Resistor_THT:R_Axial_DIN0309_L9.0mm_D3.2mm_P12.70mm_Horizontal -> Resistor_THT:R_Axial_DIN0207_L6.3mm_D2.5mm_P10.16mm_Horizontal
- moved R33 170.1 mm to (242.7, 97.8), turned to 270 degrees
- moved R32 166.1 mm to (239.4, 97.8), turned to 90 degrees
- moved J15 59.4 mm to (54.2, 138.4)
- moved R29 59.4 mm to (65.7, 145.4)
- moved R28 36.7 mm to (88.5, 145.7)
- moved R30 36.7 mm to (65.7, 142.2)
- moved R12 35.8 mm to (198.0, 95.0), turned to 90 degrees
- moved R13 23.1 mm to (193.9, 95.0)
- moved R14 22.6 mm to (202.6, 95.0), turned to 90 degrees
- moved C4 18.9 mm to (134.9, 68.7)
- moved C5 18.9 mm to (125.3, 68.7)
- moved C2 17.6 mm to (244.9, 69.3)
- moved C6 17.2 mm to (154.1, 71.2)
- moved C7 17.2 mm to (145.2, 71.2)
- moved J18 14.5 mm to (54.9, 96.1)
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- renumbered J14 to J10, J5 to J16, J6 to J17, J7 to J18, J8 to J19, J19 to J6, J11 to J7, J12 to J8, J13 to J9, R20 to R15, R21 to R16, R22 to R17, R23 to R18, R24 to R19, R25 to R20, R26 to R21, R27 to R22
Connections:
- net -12V renamed -15V
- C10 pad 2: +12V -> +15V
- C11 pad 1: +12V -> +15V
- C12 pad 2: +12V -> +15V
- C13 pad 1: +12V -> +15V
- C14 pad 2: +12V -> +15V
- C15 pad 1: +12V -> +15V
- J10 pad 5: +12V -> +15V
- J15 pad 1: /Gate8 -> /Gate5
- J15 pad 2: /Source7 -> /Source5
- J15 pad 5: +12V -> +15V
- J15 pad 6: /PWM8 -> /PWM5
- J6 pad 1: +12V -> +15V
- J7 pad 5: +12V -> +15V
- J8 pad 5: +12V -> +15V
- J9 pad 5: +12V -> +15V
- R11 pad 1: Net-(R11-Pad1) -> Net-(JP5-Pad1)
- R12 pad 2: Net-(R11-Pad1) -> /VtapOut
- R13 pad 1: Net-(JP5-Pad1) -> Net-(R13-Pad1)
- R15 pad 1: +12V -> +15V
- R16 pad 1: +12V -> +15V
- R17 pad 1: +12V -> +15V
- R18 pad 1: +12V -> +15V
- R19 pad 1: +12V -> +15V
- R20 pad 1: +12V -> +15V
- R21 pad 1: +12V -> +15V
- R22 pad 1: +12V -> +15V
- R28 pad 1: +12V -> +15V
- R28 pad 2: /PWM8 -> /PWM6
- R29 pad 1: +12V -> +15V
- R29 pad 2: /PWM8 -> /PWM5
- R30 pad 1: +12V -> +15V
- R30 pad 2: /PWM7 -> /PWM5
- R31 pad 1: Net-(R36-Pad1) -> Net-(R31-Pad1)
- R32 pad 1: +12V -> /Vm_LTSP_25-NP
- R32 pad 2: /PWM6 -> Net-(R31-Pad1)
- R33 pad 1: +12V -> GNDREF
- R33 pad 2: /PWM6 -> /Vm_LTSP_25-NP
- U1 pad 5: +12V -> +15V
- U2 pad 1: Net-(R17-Pad1) -> Net-(R13-Pad1)
- U2 pad 5: +12V -> +15V
- U3 pad 1: Net-(R19-Pad1) -> Net-(R14-Pad1)
- U3 pad 5: +12V -> +15V
- U4 pad 1: /Source1 -> Net-(L1-Pad1)
- U4 pad 4: Net-(L1-Pad1) -> /Source1
- U4 pad 8: Net-(R36-Pad1) -> Net-(R31-Pad1)
Routing:
- net +12V: track 494.7 -> 0.00 mm, vias 11 -> 0
- net +15V: track 0.00 -> 490.5 mm, vias 0 -> 11
- net /Source2: track 156.9 -> 115.3 mm
- net Net-(R36-Pad1): track 32.8 -> 0.00 mm
- net /VtapOut: track 167.8 -> 199.3 mm
- net Net-(R31-Pad1): track 0.00 -> 31.1 mm
- net GNDREF: track 377.6 -> 347.8 mm
- net /Vboost+: track 237.6 -> 264.9 mm
- net NEUT: track 427.6 -> 405.3 mm
- net Net-(J4-Pad1): track 306.7 -> 284.9 mm
- net /Vm_LTSP_25-NP: track 86.2 -> 107.6 mm
- net /Source3: track 251.9 -> 271.8 mm
- net Net-(R14-Pad1): track 8.67 -> 28.0 mm
- net /Source7: track 284.8 -> 266.7 mm
- net Net-(R11-Pad1): track 17.3 -> 0.00 mm
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Other:
- board size 308.6 x 115.6 mm -> 280.3 x 115.6 mm
- board text added: "+15"
- board text added: "-15"
- board text removed: "+12"
- board text removed: "-12"
